Commit message: renaming use_mock_hw to use_mock_hardware

File: kuka_kr5_support/urdf/kr5_arc.xacro (robot description, xacro)
@@ -5,5 +5,5 @@
   <xacro:include filename="$(find kuka_kr5_support)/urdf/kr5_arc_macro.xacro" />
   <xacro:include filename="$(find kuka_resources)/urdf/common_macro.ros2_control.xacro"/>
-  <xacro:kr5_arc_macro name="kr5_arc_mock" prefix="$(arg prefix)" use_mock_hw="$(arg use_mock_hw)" use_mock_sensor_commands="$(arg use_mock_sensor_commands)"/>
+  <xacro:kr5_arc_macro name="kr5_arc_mock" prefix="$(arg prefix)" use_mock_hardware="$(arg use_mock_hardware)" use_mock_sensor_commands="$(arg use_mock_sensor_commands)"/>
   <xacro:kuka_kr5_arc prefix=""/>
 </robot>

File: kuka_resources/urdf/common_macro.ros2_control.xacro (robot description, xacro)
@@ -1,8 +1,8 @@
 <?xml version="1.0"?>
 <robot xmlns:xacro="http://www.ros.org/wiki/xacro">
-  <xacro:macro name="kr5_arc_macro" params="name prefix use_mock_hw:=^|false use_mock_sensor_commands:=^|false">
+  <xacro:macro name="kr5_arc_macro" params="name prefix use_mock_hardware:=^|false use_mock_sensor_commands:=^|false">
     <ros2_control name="${name}" type="system">
       <hardware>
-        <xacro:if value="${use_mock_hw}">
+        <xacro:if value="${use_mock_hardware}">
           <plugin>mock_components/GenericSystem</plugin>
           <param name="mock_sensor_commands">${use_mock_sensor_commands}</param>

Commit message: removing use_mock_sensor_commands

File: kuka_kr5_support/urdf/kr5_arc.xacro (robot description, xacro)
@@ -5,5 +5,5 @@
   <xacro:include filename="$(find kuka_kr5_support)/urdf/kr5_arc_macro.xacro" />
   <xacro:include filename="$(find kuka_resources)/urdf/common_macro.ros2_control.xacro"/>
-  <xacro:kr5_arc_macro name="kr5_arc_mock" prefix="$(arg prefix)" use_mock_hardware="$(arg use_mock_hardware)" use_mock_sensor_commands="$(arg use_mock_sensor_commands)"/>
+  <xacro:kr5_arc_macro name="kr5_arc_mock" prefix="$(arg prefix)" use_mock_hardware="$(arg use_mock_hardware)"/>
   <xacro:kuka_kr5_arc prefix=""/>
 </robot>

File: kuka_resources/urdf/common_macro.ros2_control.xacro (robot description, xacro)
@@ -1,10 +1,9 @@
 <?xml version="1.0"?>
 <robot xmlns:xacro="http://www.ros.org/wiki/xacro">
-  <xacro:macro name="kr5_arc_macro" params="name prefix use_mock_hardware:=^|false use_mock_sensor_commands:=^|false">
+  <xacro:macro name="kr5_arc_macro" params="name prefix use_mock_hardware:=^|false">
     <ros2_control name="${name}" type="system">
       <hardware>
         <xacro:if value="${use_mock_hardware}">
           <plugin>mock_components/GenericSystem</plugin>
-          <param name="mock_sensor_commands">${use_mock_sensor_commands}</param>
         </xacro:if>
       </hardware>

Commit message: creating common ros2_control macro

File: kuka_kr5_support/urdf/kr5_arc.xacro (robot description, xacro)
@@ -5,5 +5,5 @@
   <xacro:include filename="$(find kuka_kr5_support)/urdf/kr5_arc_macro.xacro" />
   <xacro:include filename="$(find kuka_resources)/urdf/common_macro.ros2_control.xacro"/>
-  <xacro:kr5_arc_macro name="kr5_arc_mock" prefix="$(arg prefix)" use_mock_hardware="$(arg use_mock_hardware)"/>
+  <xacro:kuka_common_ros2_control_macro name="kr5_arc_mock" prefix="$(arg prefix)" use_mock_hardware="$(arg use_mock_hardware)"/>
   <xacro:kuka_kr5_arc prefix=""/>
 </robot>

File: kuka_resources/urdf/common_macro.ros2_control.xacro (robot description, xacro)
@@ -1,5 +1,5 @@
 <?xml version="1.0"?>
 <robot xmlns:xacro="http://www.ros.org/wiki/xacro">
-  <xacro:macro name="kr5_arc_macro" params="name prefix use_mock_hardware:=^|false">
+  <xacro:macro name="kuka_common_ros2_control_macro" params="name prefix use_mock_hardware:=^|false">
     <ros2_control name="${name}" type="system">
       <hardware>
