Commit message: Port to ROS 2 rolling (#2)
Co-authored-by: Dr. Denis <denis@stoglrobotics.de>

File: kuka_kr10_support/urdf/kr10r1100sixx.xacro (robot description, xacro)
@@ -1,5 +1,9 @@
 <?xml version="1.0"?>
 <robot name="kuka_kr10r1100sixx" xmlns:xacro="http://wiki.ros.org/xacro">
+  <xacro:arg name="prefix" default="" />
+  <xacro:arg name="use_mock_hardware" default="false" />
   <xacro:include filename="$(find kuka_kr10_support)/urdf/kr10r1100sixx_macro.xacro" />
+  <xacro:include filename="$(find kuka_resources)/urdf/common_macro.ros2_control.xacro"/>
+  <xacro:kuka_common_ros2_control_macro name="kr10r1100sixx_mock" prefix="$(arg prefix)" use_mock_hardware="$(arg use_mock_hardware)"/>
   <xacro:kuka_kr10r1100sixx prefix=""/>
 </robot>

File: kuka_kr10_support/urdf/kr10r1420.xacro (robot description, xacro)
@@ -1,5 +1,9 @@
 <?xml version="1.0"?>
 <robot name="kuka_kr10r1420" xmlns:xacro="http://wiki.ros.org/xacro">
+  <xacro:arg name="prefix" default="" />
+  <xacro:arg name="use_mock_hardware" default="false" />
   <xacro:include filename="$(find kuka_kr10_support)/urdf/kr10r1420_macro.xacro" />
+  <xacro:include filename="$(find kuka_resources)/urdf/common_macro.ros2_control.xacro"/>
+  <xacro:kuka_common_ros2_control_macro name="kr10r1420_mock" prefix="$(arg prefix)" use_mock_hardware="$(arg use_mock_hardware)"/>
   <xacro:kuka_kr10r1420 prefix=""/>
 </robot>

File: kuka_kr10_support/urdf/kr10r900_2.xacro (robot description, xacro)
@@ -1,5 +1,9 @@
 <?xml version="1.0"?>
 <robot name="kuka_kr10r900_2" xmlns:xacro="http://wiki.ros.org/xacro">
+  <xacro:arg name="prefix" default="" />
+  <xacro:arg name="use_mock_hardware" default="false" />
   <xacro:include filename="$(find kuka_kr10_support)/urdf/kr10r900_2_macro.xacro" />
+  <xacro:include filename="$(find kuka_resources)/urdf/common_macro.ros2_control.xacro"/>
+  <xacro:kuka_common_ros2_control_macro name="kr10r900_2_mock" prefix="$(arg prefix)" use_mock_hardware="$(arg use_mock_hardware)"/>
   <xacro:kuka_kr10r900_2 prefix=""/>
 </robot>

File: kuka_kr10_support/urdf/kr10r900_2_macro.xacro (robot description, xacro)
@@ -148,7 +148,12 @@
       <child link="${prefix}link_6"/>
       <axis xyz="-1 0 0"/>
-      <limit effort="0" lower="${radians(-350)}" upper="${radians(350)}" velocity="${radians(433)}"/>
+      <limit effort="0" lower="${radians(-350)}" upper="${radians(350)}" velocity="${radians(492)}"/>
     </joint>
-    <!-- ROS-Industrial 'base' frame: base_link to KUKA $ROBROOT coordinate system transform -->
+    <joint name="${prefix}joint_a6-flange" type="fixed">
+      <parent link="${prefix}link_6"/>
+      <child link="${prefix}flange"/>
+      <origin xyz="0 0 0" rpy="0 0 0"/>
+    </joint>
+    <!-- ROS-Industrial 'base'- frame base_link to KUKA $ROBROOT coordinate system transform -->
     <link name="${prefix}base" />
     <joint name="${prefix}base_link-base" type="fixed">
@@ -157,5 +162,5 @@
       <child link="${prefix}base"/>
     </joint>
-    <!-- ROS-Industrial 'flange' frame: attachment point for EEF models -->
+    <!-- ROS-Industrial 'flange' - frame attachment point for EEF models -->
     <link name="${prefix}flange" />
     <joint name="${prefix}joint_6-flange" type="fixed">
@@ -164,5 +169,5 @@
       <child link="${prefix}flange" />
     </joint>
-    <!-- ROS-Industrial 'tool0' frame: all-zeros tool frame -->
+    <!-- ROS-Industrial 'tool0' - frame all-zeros tool frame -->
     <!-- This frame corresponds to the $FLANGE coordinate system in KUKA KRC controllers. -->
     <link name="${prefix}tool0"/>

File: kuka_kr120_support/urdf/kr120r2500pro.xacro (robot description, xacro)
@@ -2,5 +2,9 @@
 <!--Generates a urdf from the macro in kr120r2500pro_macro.xacro -->
 <robot name="kuka_kr120r2500pro" xmlns:xacro="http://wiki.ros.org/xacro">
+  <xacro:arg name="prefix" default="" />
+  <xacro:arg name="use_mock_hardware" default="false" />
     <xacro:include filename="$(find kuka_kr120_support)/urdf/kr120r2500pro_macro.xacro" />
+    <xacro:include filename="$(find kuka_resources)/urdf/common_macro.ros2_control.xacro"/>
+    <xacro:kuka_common_ros2_control_macro name="kr120r2500pro_mock" prefix="$(arg prefix)" use_mock_hardware="$(arg use_mock_hardware)"/>
     <xacro:kuka_kr120r2500pro prefix=""/>
 </robot>

File: kuka_kr150_support/urdf/kr150_2.xacro (robot description, xacro)
@@ -1,5 +1,9 @@
 <?xml version="1.0"?>
 <robot name="kuka_kr150_2" xmlns:xacro="http://wiki.ros.org/xacro">
+  <xacro:arg name="prefix" default="" />
+  <xacro:arg name="use_mock_hardware" default="false" />
   <xacro:include filename="$(find kuka_kr150_support)/urdf/kr150_2_macro.xacro" />
+  <xacro:include filename="$(find kuka_resources)/urdf/common_macro.ros2_control.xacro"/>
+  <xacro:kuka_common_ros2_control_macro name="kr150_2_mock" prefix="$(arg prefix)" use_mock_hardware="$(arg use_mock_hardware)"/>
   <xacro:kuka_kr150_2 prefix=""/>
 </robot>

File: kuka_kr150_support/urdf/kr150r3100_2.xacro (robot description, xacro)
@@ -1,5 +1,9 @@
 <?xml version="1.0"?>
 <robot name="kuka_kr150r3100_2" xmlns:xacro="http://wiki.ros.org/xacro">
+  <xacro:arg name="prefix" default="" />
+  <xacro:arg name="use_mock_hardware" default="false" />
   <xacro:include filename="$(find kuka_kr150_support)/urdf/kr150r3100_2_macro.xacro" />
+  <xacro:include filename="$(find kuka_resources)/urdf/common_macro.ros2_control.xacro"/>
+  <xacro:kuka_common_ros2_control_macro name="kr150r3100_2_mock" prefix="$(arg prefix)" use_mock_hardware="$(arg use_mock_hardware)"/>
   <xacro:kuka_kr150r3100_2 prefix=""/>
 </robot>

File: kuka_kr16_support/urdf/kr16_2.xacro (robot description, xacro)
@@ -2,5 +2,9 @@
 <!--Generates a urdf from the macro in kr16_2_macro.xacro -->
 <robot name="kuka_kr16_2" xmlns:xacro="http://wiki.ros.org/xacro">
+  <xacro:arg name="prefix" default="" />
+  <xacro:arg name="use_mock_hardware" default="false" />
   <xacro:include filename="$(find kuka_kr16_support)/urdf/kr16_2_macro.xacro" />
+  <xacro:include filename="$(find kuka_resources)/urdf/common_macro.ros2_control.xacro"/>
+  <xacro:kuka_common_ros2_control_macro name="kr16_2_mock" prefix="$(arg prefix)" use_mock_hardware="$(arg use_mock_hardware)"/>
   <xacro:kuka_kr16_2 prefix=""/>
 </robot>

File: kuka_kr210_support/urdf/kr210l150.xacro (robot description, xacro)
@@ -1,5 +1,9 @@
 <?xml version="1.0" ?>
 <robot name="kuka_kr210" xmlns:xacro="http://wiki.ros.org/xacro">
+  <xacro:arg name="prefix" default="" />
+  <xacro:arg name="use_mock_hardware" default="false" />
   <xacro:include filename="$(find kuka_kr210_support)/urdf/kr210l150_macro.xacro"/>
+  <xacro:include filename="$(find kuka_resources)/urdf/common_macro.ros2_control.xacro"/>
+  <xacro:kuka_common_ros2_control_macro name="kr210l150_mock" prefix="$(arg prefix)" use_mock_hardware="$(arg use_mock_hardware)"/>
   <xacro:kuka_kr210l150 prefix=""/>
 </robot>

File: kuka_kr5_support/urdf/kr5_arc.xacro (robot description, xacro)
@@ -1,5 +1,9 @@
 <?xml version="1.0"?>
 <robot name="kuka_kr5_arc" xmlns:xacro="http://wiki.ros.org/xacro">
+  <xacro:arg name="prefix" default="" />
+  <xacro:arg name="use_mock_hardware" default="false" />
   <xacro:include filename="$(find kuka_kr5_support)/urdf/kr5_arc_macro.xacro" />
+  <xacro:include filename="$(find kuka_resources)/urdf/common_macro.ros2_control.xacro"/>
+  <xacro:kuka_common_ros2_control_macro name="kr5_arc_mock" prefix="$(arg prefix)" use_mock_hardware="$(arg use_mock_hardware)"/>
   <xacro:kuka_kr5_arc prefix=""/>
 </robot>

File: kuka_lbr_iiwa_support/urdf/lbr_iiwa_14_r820.xacro (robot description, xacro)
@@ -1,5 +1,9 @@
 <?xml version="1.0" ?>
 <robot name="kuka_lbr_iiwa_14_r820" xmlns:xacro="http://wiki.ros.org/xacro">
+  <xacro:arg name="prefix" default="" />
+  <xacro:arg name="use_mock_hardware" default="false" />
   <xacro:include filename="$(find kuka_lbr_iiwa_support)/urdf/lbr_iiwa_14_r820_macro.xacro"/>
+  <xacro:include filename="$(find kuka_lbr_iiwa_support)/urdf/kuka_lbr_iiwa_macro.ros2_control.xacro"/>
+  <xacro:kuka_common_ros2_control_macro name="lbr_iiwa_14_r820_mock" prefix="$(arg prefix)" use_mock_hardware="$(arg use_mock_hardware)"/>
   <xacro:kuka_lbr_iiwa_14_r820 prefix=""/>
 </robot>
