Commit message: all working except kr5

File: kuka_kr10_support/urdf/kr10r1100sixx.xacro (robot description, xacro)
@@ -3,7 +3,24 @@
   <xacro:arg name="prefix" default="" />
   <xacro:arg name="use_mock_hardware" default="false" />
+  <xacro:arg name="mock_sensor_commands" default="false" />
+  <xacro:arg name="sim_gazebo_classic" default="false" />
+  <xacro:arg name="sim_gazebo" default="false" />
+  <xacro:arg name="simulation_controllers" default="" />
   <xacro:include filename="$(find kuka_kr10_support)/urdf/kr10r1100sixx_macro.xacro" />
-  <xacro:include filename="$(find kuka_resources)/urdf/common_macro.ros2_control.xacro"/>
-  <xacro:kuka_common_ros2_control_macro name="kr10r1100sixx_mock" prefix="$(arg prefix)" use_mock_hardware="$(arg use_mock_hardware)"/>
-  <xacro:kuka_kr10r1100sixx prefix=""/>
+  <xacro:include filename="$(find kuka_resources)/urdf/common_sim_macro.ros2_control.xacro"/>
+   <!-- create link fixed to the "world" -->
+  <link name="world" />
+  <!-- Load robot's macro with parameters -->
+  <!-- set prefix if multiple robots are used -->
+  <xacro:kr10r1100sixx prefix="$(arg prefix)" parent="world" >
+    <origin xyz="0 0 0" rpy="0 0 0" />          <!-- position robot in the world -->
+  </xacro:kr10r1100sixx>
+  <xacro:common_macro_ros2_control_sim
+    name="kr10r1100sixx"
+    prefix="$(arg prefix)"
+    use_mock_hardware="$(arg use_mock_hardware)"
+    mock_sensor_commands="$(arg mock_sensor_commands)"
+    sim_gazebo_classic="$(arg sim_gazebo_classic)"
+    sim_gazebo="$(arg sim_gazebo)"
+    simulation_controllers="$(arg simulation_controllers)" />
 </robot>

File: kuka_kr10_support/urdf/kr10r1420.xacro (robot description, xacro)
@@ -3,7 +3,24 @@
   <xacro:arg name="prefix" default="" />
   <xacro:arg name="use_mock_hardware" default="false" />
+  <xacro:arg name="mock_sensor_commands" default="false" />
+  <xacro:arg name="sim_gazebo_classic" default="false" />
+  <xacro:arg name="sim_gazebo" default="false" />
+  <xacro:arg name="simulation_controllers" default="" />
   <xacro:include filename="$(find kuka_kr10_support)/urdf/kr10r1420_macro.xacro" />
-  <xacro:include filename="$(find kuka_resources)/urdf/common_macro.ros2_control.xacro"/>
-  <xacro:kuka_common_ros2_control_macro name="kr10r1420_mock" prefix="$(arg prefix)" use_mock_hardware="$(arg use_mock_hardware)"/>
-  <xacro:kuka_kr10r1420 prefix=""/>
+  <xacro:include filename="$(find kuka_resources)/urdf/common_sim_macro.ros2_control.xacro"/>
+   <!-- create link fixed to the "world" -->
+  <link name="world" />
+  <!-- Load robot's macro with parameters -->
+  <!-- set prefix if multiple robots are used -->
+  <xacro:kr10r1420 prefix="$(arg prefix)" parent="world" >
+    <origin xyz="0 0 0" rpy="0 0 0" />          <!-- position robot in the world -->
+  </xacro:kr10r1420>
+  <xacro:common_macro_ros2_control_sim
+    name="kr10r1420"
+    prefix="$(arg prefix)"
+    use_mock_hardware="$(arg use_mock_hardware)"
+    mock_sensor_commands="$(arg mock_sensor_commands)"
+    sim_gazebo_classic="$(arg sim_gazebo_classic)"
+    sim_gazebo="$(arg sim_gazebo)"
+    simulation_controllers="$(arg simulation_controllers)" />
 </robot>

File: kuka_kr10_support/urdf/kr10r900_2.xacro (robot description, xacro)
@@ -3,7 +3,24 @@
   <xacro:arg name="prefix" default="" />
   <xacro:arg name="use_mock_hardware" default="false" />
+  <xacro:arg name="mock_sensor_commands" default="false" />
+  <xacro:arg name="sim_gazebo_classic" default="false" />
+  <xacro:arg name="sim_gazebo" default="false" />
+  <xacro:arg name="simulation_controllers" default="" />
   <xacro:include filename="$(find kuka_kr10_support)/urdf/kr10r900_2_macro.xacro" />
-  <xacro:include filename="$(find kuka_resources)/urdf/common_macro.ros2_control.xacro"/>
-  <xacro:kuka_common_ros2_control_macro name="kr10r900_2_mock" prefix="$(arg prefix)" use_mock_hardware="$(arg use_mock_hardware)"/>
-  <xacro:kuka_kr10r900_2 prefix=""/>
+  <xacro:include filename="$(find kuka_resources)/urdf/common_sim_macro.ros2_control.xacro"/>
+   <!-- create link fixed to the "world" -->
+  <link name="world" />
+  <!-- Load robot's macro with parameters -->
+  <!-- set prefix if multiple robots are used -->
+  <xacro:kr10r900_2 prefix="$(arg prefix)" parent="world" >
+    <origin xyz="0 0 0" rpy="0 0 0" />          <!-- position robot in the world -->
+  </xacro:kr10r900_2>
+  <xacro:common_macro_ros2_control_sim
+    name="kr10r900_2"
+    prefix="$(arg prefix)"
+    use_mock_hardware="$(arg use_mock_hardware)"
+    mock_sensor_commands="$(arg mock_sensor_commands)"
+    sim_gazebo_classic="$(arg sim_gazebo_classic)"
+    sim_gazebo="$(arg sim_gazebo)"
+    simulation_controllers="$(arg simulation_controllers)" />
 </robot>

File: kuka_kr120_support/urdf/kr120r2500pro.xacro (robot description, xacro)
@@ -4,7 +4,24 @@
   <xacro:arg name="prefix" default="" />
   <xacro:arg name="use_mock_hardware" default="false" />
+  <xacro:arg name="mock_sensor_commands" default="false" />
+  <xacro:arg name="sim_gazebo_classic" default="false" />
+  <xacro:arg name="sim_gazebo" default="false" />
+  <xacro:arg name="simulation_controllers" default="" />
     <xacro:include filename="$(find kuka_kr120_support)/urdf/kr120r2500pro_macro.xacro" />
-    <xacro:include filename="$(find kuka_resources)/urdf/common_macro.ros2_control.xacro"/>
-    <xacro:kuka_common_ros2_control_macro name="kr120r2500pro_mock" prefix="$(arg prefix)" use_mock_hardware="$(arg use_mock_hardware)"/>
-    <xacro:kuka_kr120r2500pro prefix=""/>
+  <xacro:include filename="$(find kuka_resources)/urdf/common_sim_macro.ros2_control.xacro"/>
+   <!-- create link fixed to the "world" -->
+  <link name="world" />
+  <!-- Load robot's macro with parameters -->
+  <!-- set prefix if multiple robots are used -->
+  <xacro:kr120r2500pro prefix="$(arg prefix)" parent="world" >
+    <origin xyz="0 0 0" rpy="0 0 0" />          <!-- position robot in the world -->
+  </xacro:kr120r2500pro>
+  <xacro:common_macro_ros2_control_sim
+    name="kr120r2500pro"
+    prefix="$(arg prefix)"
+    use_mock_hardware="$(arg use_mock_hardware)"
+    mock_sensor_commands="$(arg mock_sensor_commands)"
+    sim_gazebo_classic="$(arg sim_gazebo_classic)"
+    sim_gazebo="$(arg sim_gazebo)"
+    simulation_controllers="$(arg simulation_controllers)" />
 </robot>

File: kuka_kr150_support/urdf/kr150_2.xacro (robot description, xacro)
@@ -3,7 +3,24 @@
   <xacro:arg name="prefix" default="" />
   <xacro:arg name="use_mock_hardware" default="false" />
+  <xacro:arg name="mock_sensor_commands" default="false" />
+  <xacro:arg name="sim_gazebo_classic" default="false" />
+  <xacro:arg name="sim_gazebo" default="false" />
+  <xacro:arg name="simulation_controllers" default="" />
   <xacro:include filename="$(find kuka_kr150_support)/urdf/kr150_2_macro.xacro" />
-  <xacro:include filename="$(find kuka_resources)/urdf/common_macro.ros2_control.xacro"/>
-  <xacro:kuka_common_ros2_control_macro name="kr150_2_mock" prefix="$(arg prefix)" use_mock_hardware="$(arg use_mock_hardware)"/>
-  <xacro:kuka_kr150_2 prefix=""/>
+  <xacro:include filename="$(find kuka_resources)/urdf/common_sim_macro.ros2_control.xacro"/>
+   <!-- create link fixed to the "world" -->
+  <link name="world" />
+  <!-- Load robot's macro with parameters -->
+  <!-- set prefix if multiple robots are used -->
+  <xacro:kr150_2 prefix="$(arg prefix)" parent="world" >
+    <origin xyz="0 0 0" rpy="0 0 0" />          <!-- position robot in the world -->
+  </xacro:kr150_2>
+  <xacro:common_macro_ros2_control_sim
+    name="kr150_2"
+    prefix="$(arg prefix)"
+    use_mock_hardware="$(arg use_mock_hardware)"
+    mock_sensor_commands="$(arg mock_sensor_commands)"
+    sim_gazebo_classic="$(arg sim_gazebo_classic)"
+    sim_gazebo="$(arg sim_gazebo)"
+    simulation_controllers="$(arg simulation_controllers)" />
 </robot>

File: kuka_kr150_support/urdf/kr150r3100_2.xacro (robot description, xacro)
@@ -3,7 +3,24 @@
   <xacro:arg name="prefix" default="" />
   <xacro:arg name="use_mock_hardware" default="false" />
+  <xacro:arg name="mock_sensor_commands" default="false" />
+  <xacro:arg name="sim_gazebo_classic" default="false" />
+  <xacro:arg name="sim_gazebo" default="false" />
+  <xacro:arg name="simulation_controllers" default="" />
   <xacro:include filename="$(find kuka_kr150_support)/urdf/kr150r3100_2_macro.xacro" />
-  <xacro:include filename="$(find kuka_resources)/urdf/common_macro.ros2_control.xacro"/>
-  <xacro:kuka_common_ros2_control_macro name="kr150r3100_2_mock" prefix="$(arg prefix)" use_mock_hardware="$(arg use_mock_hardware)"/>
-  <xacro:kuka_kr150r3100_2 prefix=""/>
+  <xacro:include filename="$(find kuka_resources)/urdf/common_sim_macro.ros2_control.xacro"/>
+   <!-- create link fixed to the "world" -->
+  <link name="world" />
+  <!-- Load robot's macro with parameters -->
+  <!-- set prefix if multiple robots are used -->
+  <xacro:kr150r3100_2 prefix="$(arg prefix)" parent="world" >
+    <origin xyz="0 0 0" rpy="0 0 0" />          <!-- position robot in the world -->
+  </xacro:kr150r3100_2>
+  <xacro:common_macro_ros2_control_sim
+    name="kr150r3100_2"
+    prefix="$(arg prefix)"
+    use_mock_hardware="$(arg use_mock_hardware)"
+    mock_sensor_commands="$(arg mock_sensor_commands)"
+    sim_gazebo_classic="$(arg sim_gazebo_classic)"
+    sim_gazebo="$(arg sim_gazebo)"
+    simulation_controllers="$(arg simulation_controllers)" />
 </robot>

File: kuka_kr16_support/urdf/kr16_2.xacro (robot description, xacro)
@@ -4,7 +4,24 @@
   <xacro:arg name="prefix" default="" />
   <xacro:arg name="use_mock_hardware" default="false" />
+  <xacro:arg name="mock_sensor_commands" default="false" />
+  <xacro:arg name="sim_gazebo_classic" default="false" />
+  <xacro:arg name="sim_gazebo" default="false" />
+  <xacro:arg name="simulation_controllers" default="" />
   <xacro:include filename="$(find kuka_kr16_support)/urdf/kr16_2_macro.xacro" />
-  <xacro:include filename="$(find kuka_resources)/urdf/common_macro.ros2_control.xacro"/>
-  <xacro:kuka_common_ros2_control_macro name="kr16_2_mock" prefix="$(arg prefix)" use_mock_hardware="$(arg use_mock_hardware)"/>
-  <xacro:kuka_kr16_2 prefix=""/>
+  <xacro:include filename="$(find kuka_resources)/urdf/common_sim_macro.ros2_control.xacro"/>
+   <!-- create link fixed to the "world" -->
+  <link name="world" />
+  <!-- Load robot's macro with parameters -->
+  <!-- set prefix if multiple robots are used -->
+  <xacro:kr16_2 prefix="$(arg prefix)" parent="world" >
+    <origin xyz="0 0 0" rpy="0 0 0" />          <!-- position robot in the world -->
+  </xacro:kr16_2>
+  <xacro:common_macro_ros2_control_sim
+    name="kr16_2"
+    prefix="$(arg prefix)"
+    use_mock_hardware="$(arg use_mock_hardware)"
+    mock_sensor_commands="$(arg mock_sensor_commands)"
+    sim_gazebo_classic="$(arg sim_gazebo_classic)"
+    sim_gazebo="$(arg sim_gazebo)"
+    simulation_controllers="$(arg simulation_controllers)" />
 </robot>

File: kuka_kr210_support/urdf/kr210l150.xacro (robot description, xacro)
@@ -3,7 +3,24 @@
   <xacro:arg name="prefix" default="" />
   <xacro:arg name="use_mock_hardware" default="false" />
+  <xacro:arg name="mock_sensor_commands" default="false" />
+  <xacro:arg name="sim_gazebo_classic" default="false" />
+  <xacro:arg name="sim_gazebo" default="false" />
+  <xacro:arg name="simulation_controllers" default="" />
   <xacro:include filename="$(find kuka_kr210_support)/urdf/kr210l150_macro.xacro"/>
-  <xacro:include filename="$(find kuka_resources)/urdf/common_macro.ros2_control.xacro"/>
-  <xacro:kuka_common_ros2_control_macro name="kr210l150_mock" prefix="$(arg prefix)" use_mock_hardware="$(arg use_mock_hardware)"/>
-  <xacro:kuka_kr210l150 prefix=""/>
+  <xacro:include filename="$(find kuka_resources)/urdf/common_sim_macro.ros2_control.xacro"/>
+   <!-- create link fixed to the "world" -->
+  <link name="world" />
+  <!-- Load robot's macro with parameters -->
+  <!-- set prefix if multiple robots are used -->
+  <xacro:kr210l150 prefix="$(arg prefix)" parent="world" >
+    <origin xyz="0 0 0" rpy="0 0 0" />          <!-- position robot in the world -->
+  </xacro:kr210l150>
+  <xacro:common_macro_ros2_control_sim
+    name="kr210l150"
+    prefix="$(arg prefix)"
+    use_mock_hardware="$(arg use_mock_hardware)"
+    mock_sensor_commands="$(arg mock_sensor_commands)"
+    sim_gazebo_classic="$(arg sim_gazebo_classic)"
+    sim_gazebo="$(arg sim_gazebo)"
+    simulation_controllers="$(arg simulation_controllers)" />
 </robot>

File: kuka_kr5_support/urdf/kr5_arc.xacro (robot description, xacro)
@@ -3,7 +3,24 @@
   <xacro:arg name="prefix" default="" />
   <xacro:arg name="use_mock_hardware" default="false" />
+  <xacro:arg name="mock_sensor_commands" default="false" />
+  <xacro:arg name="sim_gazebo_classic" default="false" />
+  <xacro:arg name="sim_gazebo" default="false" />
+  <xacro:arg name="simulation_controllers" default="" />
   <xacro:include filename="$(find kuka_kr5_support)/urdf/kr5_arc_macro.xacro" />
-  <xacro:include filename="$(find kuka_resources)/urdf/common_macro.ros2_control.xacro"/>
-  <xacro:kuka_common_ros2_control_macro name="kr5_arc_mock" prefix="$(arg prefix)" use_mock_hardware="$(arg use_mock_hardware)"/>
-  <xacro:kuka_kr5_arc prefix=""/>
+  <xacro:include filename="$(find kuka_resources)/urdf/common_sim_macro.ros2_control.xacro"/>
+   <!-- create link fixed to the "world" -->
+  <link name="world" />
+  <!-- Load robot's macro with parameters -->
+  <!-- set prefix if multiple robots are used -->
+  <xacro:kr5_arc prefix="$(arg prefix)" parent="world" >
+    <origin xyz="0 0 0" rpy="0 0 0" />          <!-- position robot in the world -->
+  </xacro:kr5_arc>
+  <xacro:common_macro_ros2_control_sim
+    name="kr5_arc"
+    prefix="$(arg prefix)"
+    use_mock_hardware="$(arg use_mock_hardware)"
+    mock_sensor_commands="$(arg mock_sensor_commands)"
+    sim_gazebo_classic="$(arg sim_gazebo_classic)"
+    sim_gazebo="$(arg sim_gazebo)"
+    simulation_controllers="$(arg simulation_controllers)" />
 </robot>

File: kuka_kr6_support/urdf/kr6r700sixx.xacro (robot description, xacro)
@@ -3,7 +3,24 @@
   <xacro:arg name="prefix" default="" />
   <xacro:arg name="use_mock_hardware" default="false" />
+  <xacro:arg name="mock_sensor_commands" default="false" />
+  <xacro:arg name="sim_gazebo_classic" default="false" />
+  <xacro:arg name="sim_gazebo" default="false" />
+  <xacro:arg name="simulation_controllers" default="" />
   <xacro:include filename="$(find kuka_kr6_support)/urdf/kr6r700sixx_macro.xacro"/>
-  <xacro:include filename="$(find kuka_resources)/urdf/common_macro.ros2_control.xacro"/>
-  <xacro:kuka_common_ros2_control_macro name="kr6r700sixx_mock" prefix="$(arg prefix)" use_mock_hardware="$(arg use_mock_hardware)"/>
-  <xacro:kuka_kr6r700sixx prefix=""/>
+  <xacro:include filename="$(find kuka_resources)/urdf/common_sim_macro.ros2_control.xacro"/>
+   <!-- create link fixed to the "world" -->
+  <link name="world" />
+  <!-- Load robot's macro with parameters -->
+  <!-- set prefix if multiple robots are used -->
+  <xacro:kr6r700sixx prefix="$(arg prefix)" parent="world" >
+    <origin xyz="0 0 0" rpy="0 0 0" />          <!-- position robot in the world -->
+  </xacro:kr6r700sixx>
+  <xacro:common_macro_ros2_control_sim
+    name="kr6r700sixx"
+    prefix="$(arg prefix)"
+    use_mock_hardware="$(arg use_mock_hardware)"
+    mock_sensor_commands="$(arg mock_sensor_commands)"
+    sim_gazebo_classic="$(arg sim_gazebo_classic)"
+    sim_gazebo="$(arg sim_gazebo)"
+    simulation_controllers="$(arg simulation_controllers)" />
 </robot>

File: kuka_kr6_support/urdf/kr6r700sixx_macro.xacro (robot description, xacro)
@@ -3,4 +3,5 @@
   <xacro:include filename="$(find kuka_resources)/urdf/common_constants.xacro"/>
   <xacro:include filename="$(find kuka_resources)/urdf/common_properties.xacro"/>
+  <xacro:include filename="$(find kuka_resources)/urdf/common_materials.xacro"/>
   <xacro:macro name="kr6r700sixx" params="prefix parent *origin">
     <link name="${prefix}base_link">

File: kuka_kr6_support/urdf/kr6r900_2.xacro (robot description, xacro)
@@ -3,7 +3,24 @@
   <xacro:arg name="prefix" default="" />
   <xacro:arg name="use_mock_hardware" default="false" />
+  <xacro:arg name="mock_sensor_commands" default="false" />
+  <xacro:arg name="sim_gazebo_classic" default="false" />
+  <xacro:arg name="sim_gazebo" default="false" />
+  <xacro:arg name="simulation_controllers" default="" />
   <xacro:include filename="$(find kuka_kr6_support)/urdf/kr6r900_2_macro.xacro" />
-  <xacro:include filename="$(find kuka_resources)/urdf/common_macro.ros2_control.xacro"/>
-  <xacro:kuka_common_ros2_control_macro name="kr6r900_2_mock" prefix="$(arg prefix)" use_mock_hardware="$(arg use_mock_hardware)"/>
-  <xacro:kuka_kr6r900_2 prefix=""/>
+  <xacro:include filename="$(find kuka_resources)/urdf/common_sim_macro.ros2_control.xacro"/>
+   <!-- create link fixed to the "world" -->
+  <link name="world" />
+  <!-- Load robot's macro with parameters -->
+  <!-- set prefix if multiple robots are used -->
+  <xacro:kr6r900_2 prefix="$(arg prefix)" parent="world" >
+    <origin xyz="0 0 0" rpy="0 0 0" />          <!-- position robot in the world -->
+  </xacro:kr6r900_2>
+  <xacro:common_macro_ros2_control_sim
+    name="kr6r900_2"
+    prefix="$(arg prefix)"
+    use_mock_hardware="$(arg use_mock_hardware)"
+    mock_sensor_commands="$(arg mock_sensor_commands)"
+    sim_gazebo_classic="$(arg sim_gazebo_classic)"
+    sim_gazebo="$(arg sim_gazebo)"
+    simulation_controllers="$(arg simulation_controllers)" />
 </robot>

File: kuka_kr6_support/urdf/kr6r900_2_macro.xacro (robot description, xacro)
@@ -2,6 +2,6 @@
 <robot xmlns:xacro="http://wiki.ros.org/xacro">
   <xacro:include filename="$(find kuka_resources)/urdf/common_properties.xacro"/>
+  <xacro:include filename="$(find kuka_resources)/urdf/common_materials.xacro"/>
   <xacro:macro name="kr6r900_2" params="prefix parent *origin">
-    <xacro:include filename="$(find kuka_resources)/urdf/common_materials.xacro"/>
     <link name="${prefix}base_link">
       <xacro:default_inertial/>
@@ -9,5 +9,5 @@
         <origin xyz="0 0 0" rpy="0 0 0"/>
         <geometry>
-          <mesh filename="file://$(find kuka_kr6_support)/meshes/kr10r900_2/visual/base_link.stl" />
+          <mesh filename="file://$(find kuka_kr10_support)/meshes/kr10r900_2/visual/base_link.stl" />
         </geometry>
         <xacro:material_kuka_ral_gray_aluminium />
@@ -16,5 +16,5 @@
         <origin xyz="0 0 0" rpy="0 0 0"/>
         <geometry>
-          <mesh filename="file://$(find kuka_kr6_support)/meshes/kr10r900_2/collision/base_link.stl" />
+          <mesh filename="file://$(find kuka_kr10_support)/meshes/kr10r900_2/collision/base_link.stl" />
         </geometry>
       </collision>
@@ -25,5 +25,5 @@
         <origin xyz="0 0 0" rpy="0 0 0"/>
         <geometry>
-          <mesh filename="file://$(find kuka_kr6_support)/meshes/kr10r900_2/visual/link_1.stl" />
+          <mesh filename="file://$(find kuka_kr10_support)/meshes/kr10r900_2/visual/link_1.stl" />
         </geometry>
         <xacro:material_kuka_ral_traffic_white />
@@ -32,5 +32,5 @@
         <origin xyz="0 0 0" rpy="0 0 0"/>
         <geometry>
-          <mesh filename="file://$(find kuka_kr6_support)/meshes/kr10r900_2/collision/link_1.stl" />
+          <mesh filename="file://$(find kuka_kr10_support)/meshes/kr10r900_2/collision/link_1.stl" />
         </geometry>
       </collision>
@@ -41,5 +41,5 @@
         <origin xyz="0 0 0" rpy="0 0 0"/>
         <geometry>
-          <mesh filename="file://$(find kuka_kr6_support)/meshes/kr10r900_2/visual/link_2.stl"/>
+          <mesh filename="file://$(find kuka_kr10_support)/meshes/kr10r900_2/visual/link_2.stl"/>
         </geometry>
         <xacro:material_kuka_ral_traffic_white />
@@ -48,5 +48,5 @@
         <origin xyz="0 0 0" rpy="0 0 0"/>
         <geometry>
-          <mesh filename="file://$(find kuka_kr6_support)/meshes/kr10r900_2/collision/link_2.stl" />
+          <mesh filename="file://$(find kuka_kr10_support)/meshes/kr10r900_2/collision/link_2.stl" />
         </geometry>
       </collision>
@@ -57,5 +57,5 @@
         <origin xyz="0 0 0" rpy="0 0 0"/>
         <geometry>
-          <mesh filename="file://$(find kuka_kr6_support)/meshes/kr10r900_2/visual/link_3.stl" />
+          <mesh filename="file://$(find kuka_kr10_support)/meshes/kr10r900_2/visual/link_3.stl" />
         </geometry>
         <xacro:material_kuka_ral_traffic_white />
@@ -64,5 +64,5 @@
         <origin xyz="0 0 0" rpy="0 0 0"/>
         <geometry>
-          <mesh filename="file://$(find kuka_kr6_support)/meshes/kr10r900_2/collision/link_3.stl" />
+          <mesh filename="file://$(find kuka_kr10_support)/meshes/kr10r900_2/collision/link_3.stl" />
         </geometry>
       </collision>
@@ -73,5 +73,5 @@
         <origin xyz="0 0 0" rpy="0 0 0"/>
         <geometry>
-          <mesh filename="file://$(find kuka_kr6_support)/meshes/kr10r900_2/visual/link_4.stl" />
+          <mesh filename="file://$(find kuka_kr10_support)/meshes/kr10r900_2/visual/link_4.stl" />
         </geometry>
         <xacro:material_kuka_ral_traffic_white />
@@ -80,5 +80,5 @@
         <origin xyz="0 0 0" rpy="0 0 0"/>
         <geometry>
-          <mesh filename="file://$(find kuka_kr6_support)/meshes/kr10r900_2/collision/link_4.stl" />
+          <mesh filename="file://$(find kuka_kr10_support)/meshes/kr10r900_2/collision/link_4.stl" />
         </geometry>
       </collision>
@@ -89,5 +89,5 @@
         <origin xyz="0 0 0" rpy="0 0 0"/>
         <geometry>
-          <mesh filename="file://$(find kuka_kr6_support)/meshes/kr10r900_2/visual/link_5.stl" />
+          <mesh filename="file://$(find kuka_kr10_support)/meshes/kr10r900_2/visual/link_5.stl" />
         </geometry>
         <xacro:material_kuka_ral_traffic_white />
@@ -96,5 +96,5 @@
         <origin xyz="0 0 0" rpy="0 0 0"/>
         <geometry>
-          <mesh filename="file://$(find kuka_kr6_support)/meshes/kr10r900_2/collision/link_5.stl" />
+          <mesh filename="file://$(find kuka_kr10_support)/meshes/kr10r900_2/collision/link_5.stl" />
         </geometry>
       </collision>
@@ -105,5 +105,5 @@
         <origin xyz="0 0 0" rpy="0 0 0"/>
         <geometry>
-          <mesh filename="file://$(find kuka_kr6_support)/meshes/kr10r900_2/visual/link_6.stl" />
+          <mesh filename="file://$(find kuka_kr10_support)/meshes/kr10r900_2/visual/link_6.stl" />
         </geometry>
         <xacro:material_kuka_black />
@@ -112,10 +112,8 @@
         <origin xyz="0 0 0" rpy="0 0 0"/>
         <geometry>
-          <mesh filename="file://$(find kuka_kr6_support)/meshes/kr10r900_2/collision/link_6.stl" />
+          <mesh filename="file://$(find kuka_kr10_support)/meshes/kr10r900_2/collision/link_6.stl" />
         </geometry>
       </collision>
     </link>
-    <!-- Following REP199, this frame shall be use to attach EEF or other equipment -->
-    <link name="${prefix}flange" />
     <!-- base_joint fixes base_link to the environment -->
     <joint name="${prefix}base_joint" type="fixed">
