Commit message: all working except kr5

File: kuka_kr6_support/urdf/kr6r900sixx.xacro (robot description, xacro)
@@ -3,7 +3,24 @@
   <xacro:arg name="prefix" default="" />
   <xacro:arg name="use_mock_hardware" default="false" />
+  <xacro:arg name="mock_sensor_commands" default="false" />
+  <xacro:arg name="sim_gazebo_classic" default="false" />
+  <xacro:arg name="sim_gazebo" default="false" />
+  <xacro:arg name="simulation_controllers" default="" />
   <xacro:include filename="$(find kuka_kr6_support)/urdf/kr6r900sixx_macro.xacro" />
-  <xacro:include filename="$(find kuka_resources)/urdf/common_macro.ros2_control.xacro"/>
-  <xacro:kuka_common_ros2_control_macro name="kr6r900sixx_mock" prefix="$(arg prefix)" use_mock_hardware="$(arg use_mock_hardware)"/>
-  <xacro:kuka_kr6r900sixx prefix=""/>
+  <xacro:include filename="$(find kuka_resources)/urdf/common_sim_macro.ros2_control.xacro"/>
+   <!-- create link fixed to the "world" -->
+  <link name="world" />
+  <!-- Load robot's macro with parameters -->
+  <!-- set prefix if multiple robots are used -->
+  <xacro:kr6r900sixx prefix="$(arg prefix)" parent="world" >
+    <origin xyz="0 0 0" rpy="0 0 0" />          <!-- position robot in the world -->
+  </xacro:kr6r900sixx>
+  <xacro:common_macro_ros2_control_sim
+    name="kr6r900sixx"
+    prefix="$(arg prefix)"
+    use_mock_hardware="$(arg use_mock_hardware)"
+    mock_sensor_commands="$(arg mock_sensor_commands)"
+    sim_gazebo_classic="$(arg sim_gazebo_classic)"
+    sim_gazebo="$(arg sim_gazebo)"
+    simulation_controllers="$(arg simulation_controllers)" />
 </robot>

Commit message: reverting robot name

File: kuka_kr10_support/urdf/kr10r1100sixx.xacro (robot description, xacro)
@@ -13,9 +13,9 @@
   <!-- Load robot's macro with parameters -->
   <!-- set prefix if multiple robots are used -->
-  <xacro:kr10r1100sixx prefix="$(arg prefix)" parent="world" >
+  <xacro:kuka_kr10r1100sixx prefix="$(arg prefix)" parent="world" >
     <origin xyz="0 0 0" rpy="0 0 0" />          <!-- position robot in the world -->
-  </xacro:kr10r1100sixx>
+  </xacro:kuka_kr10r1100sixx>
   <xacro:common_macro_ros2_control_sim
-    name="kr10r1100sixx"
+    name="kuka_kr10r1100sixx"
     prefix="$(arg prefix)"
     use_mock_hardware="$(arg use_mock_hardware)"

File: kuka_kr10_support/urdf/kr10r1100sixx_macro.xacro (robot description, xacro)
@@ -3,5 +3,5 @@
     <xacro:include filename="$(find kuka_resources)/urdf/common_materials.xacro"/>
     <xacro:include filename="$(find kuka_resources)/urdf/common_properties.xacro"/>
-  <xacro:macro name="kr10r1100sixx" params="prefix parent *origin">
+  <xacro:macro name="kuka_kr10r1100sixx" params="prefix parent *origin">
     <link name="${prefix}base_link">
       <xacro:default_inertial/>

File: kuka_kr10_support/urdf/kr10r1420.xacro (robot description, xacro)
@@ -13,9 +13,9 @@
   <!-- Load robot's macro with parameters -->
   <!-- set prefix if multiple robots are used -->
-  <xacro:kr10r1420 prefix="$(arg prefix)" parent="world" >
+  <xacro:kuka_kr10r1420 prefix="$(arg prefix)" parent="world" >
     <origin xyz="0 0 0" rpy="0 0 0" />          <!-- position robot in the world -->
-  </xacro:kr10r1420>
+  </xacro:kuka_kr10r1420>
   <xacro:common_macro_ros2_control_sim
-    name="kr10r1420"
+    name="kuka_kr10r1420"
     prefix="$(arg prefix)"
     use_mock_hardware="$(arg use_mock_hardware)"

File: kuka_kr10_support/urdf/kr10r1420_macro.xacro (robot description, xacro)
@@ -3,5 +3,5 @@
   <xacro:include filename="$(find kuka_resources)/urdf/common_materials.xacro"/>
   <xacro:include filename="$(find kuka_resources)/urdf/common_properties.xacro"/>
-  <xacro:macro name="kr10r1420" params="prefix parent *origin">
+  <xacro:macro name="kuka_kr10r1420" params="prefix parent *origin">
     <link name="${prefix}base_link">
       <xacro:default_inertial/>

File: kuka_kr10_support/urdf/kr10r900_2.xacro (robot description, xacro)
@@ -13,9 +13,9 @@
   <!-- Load robot's macro with parameters -->
   <!-- set prefix if multiple robots are used -->
-  <xacro:kr10r900_2 prefix="$(arg prefix)" parent="world" >
+  <xacro:kuka_kr10r900_2 prefix="$(arg prefix)" parent="world" >
     <origin xyz="0 0 0" rpy="0 0 0" />          <!-- position robot in the world -->
-  </xacro:kr10r900_2>
+  </xacro:kuka_kr10r900_2>
   <xacro:common_macro_ros2_control_sim
-    name="kr10r900_2"
+    name="kuka_kr10r900_2"
     prefix="$(arg prefix)"
     use_mock_hardware="$(arg use_mock_hardware)"

File: kuka_kr10_support/urdf/kr10r900_2_macro.xacro (robot description, xacro)
@@ -1,5 +1,5 @@
 <?xml version="1.0"?>
 <robot xmlns:xacro="http://wiki.ros.org/xacro">
-  <xacro:macro name="kr10r900_2" params="prefix parent *origin">
+  <xacro:macro name="kuka_kr10r900_2" params="prefix parent *origin">
     <xacro:include filename="$(find kuka_resources)/urdf/common_materials.xacro"/>
     <xacro:include filename="$(find kuka_resources)/urdf/common_properties.xacro"/>

File: kuka_kr120_support/urdf/kr120r2500pro.xacro (robot description, xacro)
@@ -14,9 +14,9 @@
   <!-- Load robot's macro with parameters -->
   <!-- set prefix if multiple robots are used -->
-  <xacro:kr120r2500pro prefix="$(arg prefix)" parent="world" >
+  <xacro:kuka_kr120r2500pro prefix="$(arg prefix)" parent="world" >
     <origin xyz="0 0 0" rpy="0 0 0" />          <!-- position robot in the world -->
-  </xacro:kr120r2500pro>
+  </xacro:kuka_kr120r2500pro>
   <xacro:common_macro_ros2_control_sim
-    name="kr120r2500pro"
+    name="kuka_kr120r2500pro"
     prefix="$(arg prefix)"
     use_mock_hardware="$(arg use_mock_hardware)"

File: kuka_kr120_support/urdf/kr120r2500pro_macro.xacro (robot description, xacro)
@@ -1,5 +1,5 @@
 <?xml version="1.0"?>
 <robot xmlns:xacro="http://wiki.ros.org/xacro">
-  <xacro:macro name="kr120r2500pro" params="prefix parent *origin">
+  <xacro:macro name="kuka_kr120r2500pro" params="prefix parent *origin">
     <!-- LINKS -->
     <!-- base link -->

File: kuka_kr150_support/urdf/kr150_2.xacro (robot description, xacro)
@@ -13,9 +13,9 @@
   <!-- Load robot's macro with parameters -->
   <!-- set prefix if multiple robots are used -->
-  <xacro:kr150_2 prefix="$(arg prefix)" parent="world" >
+  <xacro:kuka_kr150_2 prefix="$(arg prefix)" parent="world" >
     <origin xyz="0 0 0" rpy="0 0 0" />          <!-- position robot in the world -->
-  </xacro:kr150_2>
+  </xacro:kuka_kr150_2>
   <xacro:common_macro_ros2_control_sim
-    name="kr150_2"
+    name="kuka_kr150_2"
     prefix="$(arg prefix)"
     use_mock_hardware="$(arg use_mock_hardware)"

File: kuka_kr150_support/urdf/kr150_2_macro.xacro (robot description, xacro)
@@ -2,5 +2,5 @@
 <robot xmlns:xacro="http://wiki.ros.org/xacro">
   <xacro:include filename="$(find kuka_resources)/urdf/common_properties.xacro"/>
-  <xacro:macro name="kr150_2" params="prefix parent *origin">
+  <xacro:macro name="kuka_kr150_2" params="prefix parent *origin">
     <!-- LINKS -->
     <!-- base link -->

File: kuka_kr150_support/urdf/kr150r3100_2.xacro (robot description, xacro)
@@ -13,9 +13,9 @@
   <!-- Load robot's macro with parameters -->
   <!-- set prefix if multiple robots are used -->
-  <xacro:kr150r3100_2 prefix="$(arg prefix)" parent="world" >
+  <xacro:kuka_kr150r3100_2 prefix="$(arg prefix)" parent="world" >
     <origin xyz="0 0 0" rpy="0 0 0" />          <!-- position robot in the world -->
-  </xacro:kr150r3100_2>
+  </xacro:kuka_kr150r3100_2>
   <xacro:common_macro_ros2_control_sim
-    name="kr150r3100_2"
+    name="kuka_kr150r3100_2"
     prefix="$(arg prefix)"
     use_mock_hardware="$(arg use_mock_hardware)"

File: kuka_kr150_support/urdf/kr150r3100_2_macro.xacro (robot description, xacro)
@@ -3,5 +3,5 @@
   <xacro:include filename="$(find kuka_resources)/urdf/common_materials.xacro"/>
   <xacro:include filename="$(find kuka_resources)/urdf/common_properties.xacro"/>
-  <xacro:macro name="kr150r3100_2" params="prefix parent *origin">
+  <xacro:macro name="kuka_kr150r3100_2" params="prefix parent *origin">
     <!-- LINKS -->
     <!-- base link -->

File: kuka_kr16_support/urdf/kr16_2.xacro (robot description, xacro)
@@ -14,9 +14,9 @@
   <!-- Load robot's macro with parameters -->
   <!-- set prefix if multiple robots are used -->
-  <xacro:kr16_2 prefix="$(arg prefix)" parent="world" >
+  <xacro:kuka_kr16_2 prefix="$(arg prefix)" parent="world" >
     <origin xyz="0 0 0" rpy="0 0 0" />          <!-- position robot in the world -->
-  </xacro:kr16_2>
+  </xacro:kuka_kr16_2>
   <xacro:common_macro_ros2_control_sim
-    name="kr16_2"
+    name="kuka_kr16_2"
     prefix="$(arg prefix)"
     use_mock_hardware="$(arg use_mock_hardware)"

File: kuka_kr16_support/urdf/kr16_2_macro.xacro (robot description, xacro)
@@ -1,5 +1,5 @@
 <?xml version="1.0"?>
 <robot xmlns:xacro="http://wiki.ros.org/xacro">
-  <xacro:macro name="kr16_2" params="prefix parent *origin">
+  <xacro:macro name="kuka_kr16_2" params="prefix parent *origin">
     <!-- LINKS -->
     <!-- base link -->

File: kuka_kr210_support/urdf/kr210l150.xacro (robot description, xacro)
@@ -1,4 +1,4 @@
 <?xml version="1.0" ?>
-<robot name="kuka_kr210" xmlns:xacro="http://wiki.ros.org/xacro">
+<robot name="kuka_kr210l150" xmlns:xacro="http://wiki.ros.org/xacro">
   <xacro:arg name="prefix" default="" />
   <xacro:arg name="use_mock_hardware" default="false" />
@@ -13,9 +13,9 @@
   <!-- Load robot's macro with parameters -->
   <!-- set prefix if multiple robots are used -->
-  <xacro:kr210l150 prefix="$(arg prefix)" parent="world" >
+  <xacro:kuka_kr210l150 prefix="$(arg prefix)" parent="world" >
     <origin xyz="0 0 0" rpy="0 0 0" />          <!-- position robot in the world -->
-  </xacro:kr210l150>
+  </xacro:kuka_kr210l150>
   <xacro:common_macro_ros2_control_sim
-    name="kr210l150"
+    name="kuka_kr210l150"
     prefix="$(arg prefix)"
     use_mock_hardware="$(arg use_mock_hardware)"

File: kuka_kr210_support/urdf/kr210l150_macro.xacro (robot description, xacro)
@@ -1,5 +1,5 @@
 <?xml version="1.0"?>
 <robot xmlns:xacro="http://wiki.ros.org/xacro">
-  <xacro:macro name="kr210l150" params="prefix parent *origin">
+  <xacro:macro name="kuka_kr210l150" params="prefix parent *origin">
     <!-- links -->
     <link name="${prefix}base_link">

File: kuka_kr3_support/urdf/kr3r540.xacro (robot description, xacro)
@@ -1,4 +1,4 @@
 <?xml version="1.0" ?>
-<robot name="kr3r540" xmlns:xacro="http://wiki.ros.org/xacro">
+<robot name="kuka_kr3r540" xmlns:xacro="http://wiki.ros.org/xacro">
   <xacro:arg name="prefix" default="" />
   <xacro:arg name="use_mock_hardware" default="false" />
@@ -13,9 +13,9 @@
   <!-- Load robot's macro with parameters -->
   <!-- set prefix if multiple robots are used -->
-  <xacro:kr3r540 prefix="$(arg prefix)" parent="world" >
+  <xacro:kuka_kr3r540 prefix="$(arg prefix)" parent="world" >
     <origin xyz="0 0 0" rpy="0 0 0" />          <!-- position robot in the world -->
-  </xacro:kr3r540>
+  </xacro:kuka_kr3r540>
   <xacro:common_macro_ros2_control_sim
-    name="kr3r540"
+    name="kuka_kr3r540"
     prefix="$(arg prefix)"
     use_mock_hardware="$(arg use_mock_hardware)"

File: kuka_kr3_support/urdf/kr3r540_macro.xacro (robot description, xacro)
@@ -3,5 +3,5 @@
   <xacro:include filename="$(find kuka_resources)/urdf/common_materials.xacro"/>
   <xacro:include filename="$(find kuka_resources)/urdf/common_properties.xacro"/>
-  <xacro:macro name="kr3r540" params="prefix parent *origin">
+  <xacro:macro name="kuka_kr3r540" params="prefix parent *origin">
     <link name="${prefix}base_link">
       <xacro:default_inertial/>

File: kuka_kr5_support/urdf/kr5_arc.xacro (robot description, xacro)
@@ -13,9 +13,9 @@
   <!-- Load robot's macro with parameters -->
   <!-- set prefix if multiple robots are used -->
-  <xacro:kr5_arc prefix="$(arg prefix)" parent="world" >
+  <xacro:kuka_kr5_arc prefix="$(arg prefix)" parent="world" >
     <origin xyz="0 0 0" rpy="0 0 0" />          <!-- position robot in the world -->
-  </xacro:kr5_arc>
+  </xacro:kuka_kr5_arc>
   <xacro:common_macro_ros2_control_sim
-    name="kr5_arc"
+    name="kuka_kr5_arc"
     prefix="$(arg prefix)"
     use_mock_hardware="$(arg use_mock_hardware)"

File: kuka_kr5_support/urdf/kr5_arc_macro.xacro (robot description, xacro)
@@ -1,5 +1,5 @@
 <?xml version="1.0"?>
 <robot xmlns:xacro="http://wiki.ros.org/xacro">
-  <xacro:macro name="kr5_arc" params="prefix parent *origin">
+  <xacro:macro name="kuka_kr5_arc" params="prefix parent *origin">
     <!-- LINKS -->
     <!-- base link -->
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