Commit message: removed duplicate and adjusted

File: kuka_kr10_support/urdf/kr10r1100sixx.xacro (robot description, xacro)
@@ -8,5 +8,5 @@
   <xacro:arg name="simulation_controllers" default="" />
   <xacro:include filename="$(find kuka_kr10_support)/urdf/kr10r1100sixx_macro.xacro" />
-  <xacro:include filename="$(find kuka_resources)/urdf/common_sim_macro.ros2_control.xacro"/>
+  <xacro:include filename="$(find kuka_resources)/urdf/common_macro.ros2_control.xacro"/>
    <!-- create link fixed to the "world" -->
   <link name="world" />
@@ -16,5 +16,5 @@
     <origin xyz="0 0 0" rpy="0 0 0" />          <!-- position robot in the world -->
   </xacro:kuka_kr10r1100sixx>
-  <xacro:common_macro_ros2_control_sim
+  <xacro:kuka_common_ros2_control_macro
     name="kuka_kr10r1100sixx"
     prefix="$(arg prefix)"

File: kuka_kr10_support/urdf/kr10r1420.xacro (robot description, xacro)
@@ -8,5 +8,5 @@
   <xacro:arg name="simulation_controllers" default="" />
   <xacro:include filename="$(find kuka_kr10_support)/urdf/kr10r1420_macro.xacro" />
-  <xacro:include filename="$(find kuka_resources)/urdf/common_sim_macro.ros2_control.xacro"/>
+  <xacro:include filename="$(find kuka_resources)/urdf/common_macro.ros2_control.xacro"/>
    <!-- create link fixed to the "world" -->
   <link name="world" />
@@ -16,5 +16,5 @@
     <origin xyz="0 0 0" rpy="0 0 0" />          <!-- position robot in the world -->
   </xacro:kuka_kr10r1420>
-  <xacro:common_macro_ros2_control_sim
+  <xacro:kuka_common_ros2_control_macro
     name="kuka_kr10r1420"
     prefix="$(arg prefix)"

File: kuka_kr10_support/urdf/kr10r900_2.xacro (robot description, xacro)
@@ -8,5 +8,5 @@
   <xacro:arg name="simulation_controllers" default="" />
   <xacro:include filename="$(find kuka_kr10_support)/urdf/kr10r900_2_macro.xacro" />
-  <xacro:include filename="$(find kuka_resources)/urdf/common_sim_macro.ros2_control.xacro"/>
+  <xacro:include filename="$(find kuka_resources)/urdf/common_macro.ros2_control.xacro"/>
    <!-- create link fixed to the "world" -->
   <link name="world" />
@@ -16,5 +16,5 @@
     <origin xyz="0 0 0" rpy="0 0 0" />          <!-- position robot in the world -->
   </xacro:kuka_kr10r900_2>
-  <xacro:common_macro_ros2_control_sim
+  <xacro:kuka_common_ros2_control_macro
     name="kuka_kr10r900_2"
     prefix="$(arg prefix)"

File: kuka_kr120_support/urdf/kr120r2500pro.xacro (robot description, xacro)
@@ -9,5 +9,5 @@
   <xacro:arg name="simulation_controllers" default="" />
     <xacro:include filename="$(find kuka_kr120_support)/urdf/kr120r2500pro_macro.xacro" />
-  <xacro:include filename="$(find kuka_resources)/urdf/common_sim_macro.ros2_control.xacro"/>
+  <xacro:include filename="$(find kuka_resources)/urdf/common_macro.ros2_control.xacro"/>
    <!-- create link fixed to the "world" -->
   <link name="world" />
@@ -17,5 +17,5 @@
     <origin xyz="0 0 0" rpy="0 0 0" />          <!-- position robot in the world -->
   </xacro:kuka_kr120r2500pro>
-  <xacro:common_macro_ros2_control_sim
+  <xacro:kuka_common_ros2_control_macro
     name="kuka_kr120r2500pro"
     prefix="$(arg prefix)"

File: kuka_kr150_support/urdf/kr150_2.xacro (robot description, xacro)
@@ -8,5 +8,5 @@
   <xacro:arg name="simulation_controllers" default="" />
   <xacro:include filename="$(find kuka_kr150_support)/urdf/kr150_2_macro.xacro" />
-  <xacro:include filename="$(find kuka_resources)/urdf/common_sim_macro.ros2_control.xacro"/>
+  <xacro:include filename="$(find kuka_resources)/urdf/common_macro.ros2_control.xacro"/>
    <!-- create link fixed to the "world" -->
   <link name="world" />
@@ -16,5 +16,5 @@
     <origin xyz="0 0 0" rpy="0 0 0" />          <!-- position robot in the world -->
   </xacro:kuka_kr150_2>
-  <xacro:common_macro_ros2_control_sim
+  <xacro:kuka_common_ros2_control_macro
     name="kuka_kr150_2"
     prefix="$(arg prefix)"

File: kuka_kr150_support/urdf/kr150r3100_2.xacro (robot description, xacro)
@@ -8,5 +8,5 @@
   <xacro:arg name="simulation_controllers" default="" />
   <xacro:include filename="$(find kuka_kr150_support)/urdf/kr150r3100_2_macro.xacro" />
-  <xacro:include filename="$(find kuka_resources)/urdf/common_sim_macro.ros2_control.xacro"/>
+  <xacro:include filename="$(find kuka_resources)/urdf/common_macro.ros2_control.xacro"/>
    <!-- create link fixed to the "world" -->
   <link name="world" />
@@ -16,5 +16,5 @@
     <origin xyz="0 0 0" rpy="0 0 0" />          <!-- position robot in the world -->
   </xacro:kuka_kr150r3100_2>
-  <xacro:common_macro_ros2_control_sim
+  <xacro:kuka_common_ros2_control_macro
     name="kuka_kr150r3100_2"
     prefix="$(arg prefix)"

File: kuka_kr16_support/urdf/kr16_2.xacro (robot description, xacro)
@@ -9,5 +9,5 @@
   <xacro:arg name="simulation_controllers" default="" />
   <xacro:include filename="$(find kuka_kr16_support)/urdf/kr16_2_macro.xacro" />
-  <xacro:include filename="$(find kuka_resources)/urdf/common_sim_macro.ros2_control.xacro"/>
+  <xacro:include filename="$(find kuka_resources)/urdf/common_macro.ros2_control.xacro"/>
    <!-- create link fixed to the "world" -->
   <link name="world" />
@@ -17,5 +17,5 @@
     <origin xyz="0 0 0" rpy="0 0 0" />          <!-- position robot in the world -->
   </xacro:kuka_kr16_2>
-  <xacro:common_macro_ros2_control_sim
+  <xacro:kuka_common_ros2_control_macro
     name="kuka_kr16_2"
     prefix="$(arg prefix)"

File: kuka_kr210_support/urdf/kr210l150.xacro (robot description, xacro)
@@ -8,5 +8,5 @@
   <xacro:arg name="simulation_controllers" default="" />
   <xacro:include filename="$(find kuka_kr210_support)/urdf/kr210l150_macro.xacro"/>
-  <xacro:include filename="$(find kuka_resources)/urdf/common_sim_macro.ros2_control.xacro"/>
+  <xacro:include filename="$(find kuka_resources)/urdf/common_macro.ros2_control.xacro"/>
    <!-- create link fixed to the "world" -->
   <link name="world" />
@@ -16,5 +16,5 @@
     <origin xyz="0 0 0" rpy="0 0 0" />          <!-- position robot in the world -->
   </xacro:kuka_kr210l150>
-  <xacro:common_macro_ros2_control_sim
+  <xacro:kuka_common_ros2_control_macro
     name="kuka_kr210l150"
     prefix="$(arg prefix)"

File: kuka_kr3_support/urdf/kr3r540.xacro (robot description, xacro)
@@ -8,5 +8,5 @@
   <xacro:arg name="simulation_controllers" default="" />
   <xacro:include filename="$(find kuka_kr3_support)/urdf/kr3r540_macro.xacro"/>
-  <xacro:include filename="$(find kuka_resources)/urdf/common_sim_macro.ros2_control.xacro"/>
+  <xacro:include filename="$(find kuka_resources)/urdf/common_macro.ros2_control.xacro"/>
    <!-- create link fixed to the "world" -->
   <link name="world" />
@@ -16,5 +16,5 @@
     <origin xyz="0 0 0" rpy="0 0 0" />          <!-- position robot in the world -->
   </xacro:kuka_kr3r540>
-  <xacro:common_macro_ros2_control_sim
+  <xacro:kuka_common_ros2_control_macro
     name="kuka_kr3r540"
     prefix="$(arg prefix)"

File: kuka_kr5_support/urdf/kr5_arc.xacro (robot description, xacro)
@@ -8,5 +8,5 @@
   <xacro:arg name="simulation_controllers" default="" />
   <xacro:include filename="$(find kuka_kr5_support)/urdf/kr5_arc_macro.xacro" />
-  <xacro:include filename="$(find kuka_resources)/urdf/common_sim_macro.ros2_control.xacro"/>
+  <xacro:include filename="$(find kuka_resources)/urdf/common_macro.ros2_control.xacro"/>
    <!-- create link fixed to the "world" -->
   <link name="world" />
@@ -16,5 +16,5 @@
     <origin xyz="0 0 0" rpy="0 0 0" />          <!-- position robot in the world -->
   </xacro:kuka_kr5_arc>
-  <xacro:common_macro_ros2_control_sim
+  <xacro:kuka_common_ros2_control_macro
     name="kuka_kr5_arc"
     prefix="$(arg prefix)"

File: kuka_kr6_support/urdf/kr6r700sixx.xacro (robot description, xacro)
@@ -8,5 +8,5 @@
   <xacro:arg name="simulation_controllers" default="" />
   <xacro:include filename="$(find kuka_kr6_support)/urdf/kr6r700sixx_macro.xacro"/>
-  <xacro:include filename="$(find kuka_resources)/urdf/common_sim_macro.ros2_control.xacro"/>
+  <xacro:include filename="$(find kuka_resources)/urdf/common_macro.ros2_control.xacro"/>
    <!-- create link fixed to the "world" -->
   <link name="world" />
@@ -16,5 +16,5 @@
     <origin xyz="0 0 0" rpy="0 0 0" />          <!-- position robot in the world -->
   </xacro:kuka_kr6r700sixx>
-  <xacro:common_macro_ros2_control_sim
+  <xacro:kuka_common_ros2_control_macro
     name="kuka_kr6r700sixx"
     prefix="$(arg prefix)"

File: kuka_kr6_support/urdf/kr6r900_2.xacro (robot description, xacro)
@@ -8,5 +8,5 @@
   <xacro:arg name="simulation_controllers" default="" />
   <xacro:include filename="$(find kuka_kr6_support)/urdf/kr6r900_2_macro.xacro" />
-  <xacro:include filename="$(find kuka_resources)/urdf/common_sim_macro.ros2_control.xacro"/>
+  <xacro:include filename="$(find kuka_resources)/urdf/common_macro.ros2_control.xacro"/>
    <!-- create link fixed to the "world" -->
   <link name="world" />
@@ -16,5 +16,5 @@
     <origin xyz="0 0 0" rpy="0 0 0" />          <!-- position robot in the world -->
   </xacro:kuka_kr6r900_2>
-  <xacro:common_macro_ros2_control_sim
+  <xacro:kuka_common_ros2_control_macro
     name="kuka_kr6r900_2"
     prefix="$(arg prefix)"

File: kuka_kr6_support/urdf/kr6r900sixx.xacro (robot description, xacro)
@@ -8,5 +8,5 @@
   <xacro:arg name="simulation_controllers" default="" />
   <xacro:include filename="$(find kuka_kr6_support)/urdf/kr6r900sixx_macro.xacro" />
-  <xacro:include filename="$(find kuka_resources)/urdf/common_sim_macro.ros2_control.xacro"/>
+  <xacro:include filename="$(find kuka_resources)/urdf/common_macro.ros2_control.xacro"/>
    <!-- create link fixed to the "world" -->
   <link name="world" />
@@ -16,5 +16,5 @@
     <origin xyz="0 0 0" rpy="0 0 0" />          <!-- position robot in the world -->
   </xacro:kuka_kr6r900sixx>
-  <xacro:common_macro_ros2_control_sim
+  <xacro:kuka_common_ros2_control_macro
     name="kuka_kr6r900sixx"
     prefix="$(arg prefix)"

File: kuka_resources/urdf/common_macro.ros2_control.xacro (robot description, xacro)
@@ -1,10 +1,28 @@
 <?xml version="1.0"?>
 <robot xmlns:xacro="http://www.ros.org/wiki/xacro">
-  <xacro:macro name="kuka_common_ros2_control_macro" params="name prefix use_mock_hardware:=^|false">
+  <xacro:macro name="kuka_common_ros2_control_macro" params="
+               name
+               prefix
+               use_mock_hardware:=^|false
+               mock_sensor_commands:=^|false
+               sim_gazebo_classic:=^|false
+               sim_gazebo:=^|false
+               simulation_controllers"
+               >
     <ros2_control name="${name}" type="system">
       <hardware>
         <xacro:if value="${use_mock_hardware}">
           <plugin>mock_components/GenericSystem</plugin>
+          <param name="mock_sensor_commands">${mock_sensor_commands}</param>
         </xacro:if>
+        <xacro:if value="${sim_gazebo_classic}">
+          <plugin>gazebo_ros2_control/GazeboSystem</plugin>
+        </xacro:if>
+        <xacro:if value="${sim_gazebo}">
+          <plugin>ign_ros2_control/IgnitionSystem</plugin>
+        </xacro:if>
+        <xacro:unless value="${use_mock_hardware or sim_gazebo_classic or sim_gazebo}">
+          <plugin>robot_hardware_inteface/RobotHardwareInteface</plugin>
+        </xacro:unless>
       </hardware>
       <joint name="${prefix}joint_a1">
@@ -62,5 +80,47 @@
         </state_interface>
       </joint>
+      <sensor name="tcp_fts_sensor">            <!-- Remove/change sensors as needed -->
+        <state_interface name="fx"/>
+        <state_interface name="fy"/>
+        <state_interface name="fz"/>
+        <state_interface name="tx"/>
+        <state_interface name="ty"/>
+        <state_interface name="tz"/>
+        <param name="frame_id">tool0</param>    <!-- Change sensors as needed -->
+        <param name="min_fx">-100</param>
+        <param name="max_fx">100</param>
+        <param name="min_fy">-100</param>
+        <param name="max_fy">100</param>
+        <param name="min_fz">-200</param>
+        <param name="max_fz">200</param>
+        <param name="min_tx">-10</param>
+        <param name="max_tx">10</param>
+        <param name="min_ty">-10</param>
+        <param name="max_ty">10</param>
+        <param name="min_tz">-15</param>
+        <param name="max_tz">15</param>
+      </sensor>
     </ros2_control>
+    <xacro:if value="$(arg sim_gazebo_classic)">
+      <!-- Gazebo plugins -->
+      <gazebo reference="world">
+      </gazebo>
+      <gazebo>
+        <plugin filename="libgazebo_ros2_control.so" name="gazebo_ros2_control">
+          <parameters>${simulation_controllers}</parameters>
+        </plugin>
+      </gazebo>
+    </xacro:if>
+    <xacro:if value="$(arg sim_gazebo)">
+      <!-- Gazebo plugins -->
+      <gazebo reference="world">
+      </gazebo>
+      <gazebo>
+        <plugin filename="libign_ros2_control-system.so" name="ign_ros2_control::IgnitionROS2ControlPlugin">
+          <parameters>${simulation_controllers}</parameters>
+          <controller_manager_node_name>${prefix}controller_manager</controller_manager_node_name>
+        </plugin>
+      </gazebo>
+    </xacro:if>
   </xacro:macro>
 </robot>
