Commit message: added ignition launch for kuka_lbr and its respective files modified

File: kuka_lbr_iiwa_support/urdf/kuka_lbr_iiwa_macro.ros2_control.xacro (robot description, xacro)
@@ -1,5 +1,8 @@
 <?xml version="1.0"?>
 <robot xmlns:xacro="http://www.ros.org/wiki/xacro">
-  <xacro:macro name="kuka_common_ros2_control_macro" params="name prefix use_mock_hardware:=^|false">
+  <xacro:macro name="kuka_common_ros2_control_macro" params="
+                name
+                prefix
+                use_mock_hardware:=^|false">
     <ros2_control name="${name}" type="system">
       <hardware>

File: kuka_lbr_iiwa_support/urdf/lbr_iiwa_14_r820.xacro (robot description, xacro)
@@ -3,7 +3,24 @@
   <xacro:arg name="prefix" default="" />
   <xacro:arg name="use_mock_hardware" default="false" />
+  <xacro:arg name="mock_sensor_commands" default="false" />
+  <xacro:arg name="sim_gazebo_classic" default="false" />
+  <xacro:arg name="sim_gazebo" default="false" />
+  <xacro:arg name="simulation_controllers" default="" />
   <xacro:include filename="$(find kuka_lbr_iiwa_support)/urdf/lbr_iiwa_14_r820_macro.xacro"/>
-  <xacro:include filename="$(find kuka_lbr_iiwa_support)/urdf/kuka_lbr_iiwa_macro.ros2_control.xacro"/>
-  <xacro:kuka_common_ros2_control_macro name="lbr_iiwa_14_r820_mock" prefix="$(arg prefix)" use_mock_hardware="$(arg use_mock_hardware)"/>
-  <xacro:kuka_lbr_iiwa_14_r820 prefix=""/>
+  <xacro:include filename="$(find kuka_lbr_iiwa_support)/urdf/kuka_lbr_iiwa_sim_macro.ros2_control.xacro"/>
+   <!-- create link fixed to the "world" -->
+  <link name="world" />
+  <!-- Load robot's macro with parameters -->
+  <!-- set prefix if multiple robots are used -->
+  <xacro:kuka_lbr_iiwa_14_r820 prefix="$(arg prefix)" parent="world" >
+    <origin xyz="0 0 0" rpy="0 0 0" />          <!-- position robot in the world -->
+  </xacro:kuka_lbr_iiwa_14_r820>
+  <xacro:kuka_lbr_iiwa_ros2_control_sim
+    name="lbr_iiwa_14_r820"
+    prefix="$(arg prefix)"
+    use_mock_hardware="$(arg use_mock_hardware)"
+    mock_sensor_commands="$(arg mock_sensor_commands)"
+    sim_gazebo_classic="$(arg sim_gazebo_classic)"
+    sim_gazebo="$(arg sim_gazebo)"
+    simulation_controllers="$(arg simulation_controllers)" />
 </robot>

File: kuka_lbr_iiwa_support/urdf/lbr_iiwa_14_r820_macro.xacro (robot description, xacro)
@@ -1,11 +1,13 @@
 <?xml version="1.0"?>
 <robot xmlns:xacro="http://wiki.ros.org/xacro">
-  <xacro:macro name="kuka_lbr_iiwa_14_r820" params="prefix">
+  <xacro:include filename="$(find kuka_resources)/urdf/common_materials.xacro"/>
+  <xacro:macro name="kuka_lbr_iiwa_14_r820" params="prefix parent *origin">
     <!-- link list -->
     <link name="${prefix}base_link">
+      <xacro:default_inertial/>
       <visual>
         <origin xyz="0 0 0" rpy="0 0 0" />
         <geometry>
-          <mesh filename="package://kuka_lbr_iiwa_support/meshes/lbr_iiwa_14_r820/visual/base_link.dae" />
+          <mesh filename="file://$(find kuka_lbr_iiwa_support)/meshes/lbr_iiwa_14_r820/visual/base_link.dae" />
         </geometry>
       </visual>
@@ -13,13 +15,14 @@
         <origin xyz="0 0 0" rpy="0 0 0" />
         <geometry>
-          <mesh filename="package://kuka_lbr_iiwa_support/meshes/lbr_iiwa_14_r820/collision/base_link.stl" />
+          <mesh filename="file://$(find kuka_lbr_iiwa_support)/meshes/lbr_iiwa_14_r820/collision/base_link.stl" />
         </geometry>
       </collision>
     </link>
     <link name="${prefix}link_1">
+      <xacro:default_inertial/>
       <visual>
         <origin xyz="0 0 0" rpy="0 0 0" />
         <geometry>
-          <mesh filename="package://kuka_lbr_iiwa_support/meshes/lbr_iiwa_14_r820/visual/link_1.dae" />
+          <mesh filename="file://$(find kuka_lbr_iiwa_support)/meshes/lbr_iiwa_14_r820/visual/link_1.dae" />
         </geometry>
       </visual>
@@ -27,13 +30,14 @@
         <origin xyz="0 0 0" rpy="0 0 0" />
         <geometry>
-          <mesh filename="package://kuka_lbr_iiwa_support/meshes/lbr_iiwa_14_r820/collision/link_1.stl" />
+          <mesh filename="file://$(find kuka_lbr_iiwa_support)/meshes/lbr_iiwa_14_r820/collision/link_1.stl" />
         </geometry>
       </collision>
     </link>
     <link name="${prefix}link_2">
+      <xacro:default_inertial/>
       <visual>
         <origin xyz="0 0 0" rpy="0 0 0" />
         <geometry>
-          <mesh filename="package://kuka_lbr_iiwa_support/meshes/lbr_iiwa_14_r820/visual/link_2.dae" />
+          <mesh filename="file://$(find kuka_lbr_iiwa_support)/meshes/lbr_iiwa_14_r820/visual/link_2.dae" />
         </geometry>
       </visual>
@@ -41,13 +45,14 @@
         <origin xyz="0 0 0" rpy="0 0 0" />
         <geometry>
-          <mesh filename="package://kuka_lbr_iiwa_support/meshes/lbr_iiwa_14_r820/collision/link_2.stl" />
+          <mesh filename="file://$(find kuka_lbr_iiwa_support)/meshes/lbr_iiwa_14_r820/collision/link_2.stl" />
         </geometry>
       </collision>
     </link>
     <link name="${prefix}link_3">
+      <xacro:default_inertial/>
       <visual>
         <origin xyz="0 0 0" rpy="0 0 0" />
         <geometry>
-          <mesh filename="package://kuka_lbr_iiwa_support/meshes/lbr_iiwa_14_r820/visual/link_3.dae" />
+          <mesh filename="file://$(find kuka_lbr_iiwa_support)/meshes/lbr_iiwa_14_r820/visual/link_3.dae" />
         </geometry>
       </visual>
@@ -55,13 +60,14 @@
         <origin xyz="0 0 0" rpy="0 0 0" />
         <geometry>
-          <mesh filename="package://kuka_lbr_iiwa_support/meshes/lbr_iiwa_14_r820/collision/link_3.stl" />
+          <mesh filename="file://$(find kuka_lbr_iiwa_support)/meshes/lbr_iiwa_14_r820/collision/link_3.stl" />
         </geometry>
       </collision>
     </link>
     <link name="${prefix}link_4">
+      <xacro:default_inertial/>
       <visual>
         <origin xyz="0 0 0" rpy="0 0 0" />
         <geometry>
-          <mesh filename="package://kuka_lbr_iiwa_support/meshes/lbr_iiwa_14_r820/visual/link_4.dae" />
+          <mesh filename="file://$(find kuka_lbr_iiwa_support)/meshes/lbr_iiwa_14_r820/visual/link_4.dae" />
         </geometry>
       </visual>
@@ -69,13 +75,14 @@
         <origin xyz="0 0 0" rpy="0 0 0" />
         <geometry>
-          <mesh filename="package://kuka_lbr_iiwa_support/meshes/lbr_iiwa_14_r820/collision/link_4.stl" />
+          <mesh filename="file://$(find kuka_lbr_iiwa_support)/meshes/lbr_iiwa_14_r820/collision/link_4.stl" />
         </geometry>
       </collision>
     </link>
     <link name="${prefix}link_5">
+      <xacro:default_inertial/>
       <visual>
         <origin xyz="0 0 0" rpy="0 0 0" />
         <geometry>
-          <mesh filename="package://kuka_lbr_iiwa_support/meshes/lbr_iiwa_14_r820/visual/link_5.dae" />
+          <mesh filename="file://$(find kuka_lbr_iiwa_support)/meshes/lbr_iiwa_14_r820/visual/link_5.dae" />
         </geometry>
       </visual>
@@ -83,13 +90,14 @@
         <origin xyz="0 0 0" rpy="0 0 0" />
         <geometry>
-          <mesh filename="package://kuka_lbr_iiwa_support/meshes/lbr_iiwa_14_r820/collision/link_5.stl" />
+          <mesh filename="file://$(find kuka_lbr_iiwa_support)/meshes/lbr_iiwa_14_r820/collision/link_5.stl" />
         </geometry>
       </collision>
     </link>
     <link name="${prefix}link_6">
+      <xacro:default_inertial/>
       <visual>
         <origin xyz="0 0 0" rpy="0 0 0" />
         <geometry>
-          <mesh filename="package://kuka_lbr_iiwa_support/meshes/lbr_iiwa_14_r820/visual/link_6.dae" />
+          <mesh filename="file://$(find kuka_lbr_iiwa_support)/meshes/lbr_iiwa_14_r820/visual/link_6.dae" />
         </geometry>
       </visual>
@@ -97,13 +105,14 @@
         <origin xyz="0 0 0" rpy="0 0 0" />
         <geometry>
-          <mesh filename="package://kuka_lbr_iiwa_support/meshes/lbr_iiwa_14_r820/collision/link_6.stl" />
+          <mesh filename="file://$(find kuka_lbr_iiwa_support)/meshes/lbr_iiwa_14_r820/collision/link_6.stl" />
         </geometry>
       </collision>
     </link>
     <link name="${prefix}link_7">
+      <xacro:default_inertial/>
       <visual>
         <origin xyz="0 0 0" rpy="0 0 0" />
         <geometry>
-          <mesh filename="package://kuka_lbr_iiwa_support/meshes/lbr_iiwa_14_r820/visual/link_7.dae" />
+          <mesh filename="file://$(find kuka_lbr_iiwa_support)/meshes/lbr_iiwa_14_r820/visual/link_7.dae" />
         </geometry>
       </visual>
@@ -111,5 +120,5 @@
         <origin xyz="0 0 0" rpy="0 0 0" />
         <geometry>
-          <mesh filename="package://kuka_lbr_iiwa_support/meshes/lbr_iiwa_14_r820/collision/link_7.stl" />
+          <mesh filename="file://$(find kuka_lbr_iiwa_support)/meshes/lbr_iiwa_14_r820/collision/link_7.stl" />
         </geometry>
       </collision>
@@ -117,5 +126,10 @@
     <link name="${prefix}tool0" />
     <!-- end of link list -->
-    <!-- joint list -->
+    <!-- base_joint fixes base_link to the environment -->
+    <joint name="${prefix}base_joint" type="fixed">
+      <xacro:insert_block name="origin" />
+      <parent link="${parent}" />
+      <child link="${prefix}base_link" />
+    </joint>
     <joint name="${prefix}joint_a1" type="revolute">
       <origin xyz="0 0 0" rpy="0 0 0" />
