Commit message: added general macro name

File: kuka_resources/urdf/common_sim_macro.ros2_control.xacro (robot description, xacro)
@@ -1,5 +1,5 @@
 <?xml version="1.0" encoding="UTF-8"?>
 <robot xmlns:xacro="http://wiki.ros.org/xacro">
-  <xacro:macro name="kr3r540_ros2_control" params="
+  <xacro:macro name="common_macro_ros2_control_sim" params="
                name
                prefix
