Commit message: added inertial tag

File: kuka_resources/urdf/common_materials.xacro (robot description, xacro)
@@ -167,3 +167,10 @@
     </material>
   </xacro:macro>
+  <xacro:macro name="default_inertial">
+    <inertial>
+      <mass value="0.01"/>
+      <origin xyz="0 0 0"/>
+      <inertia ixx="0.001" ixy="0.0" ixz="0.0" iyy="0.001" iyz="0.0" izz="0.001" />
+    </inertial>
+  </xacro:macro>
 </robot>

Commit message: added a seperate xacro for default inertial

File: kuka_resources/urdf/common_materials.xacro (robot description, xacro)
@@ -167,10 +167,3 @@
     </material>
   </xacro:macro>
-  <xacro:macro name="default_inertial">
-    <inertial>
-      <mass value="0.01"/>
-      <origin xyz="0 0 0"/>
-      <inertia ixx="0.001" ixy="0.0" ixz="0.0" iyy="0.001" iyz="0.0" izz="0.001" />
-    </inertial>
-  </xacro:macro>
 </robot>
