Commit message: extended macros and xacro

File: kuka_kr3_support/urdf/kr3r540.xacro (robot description, xacro)
@@ -1,9 +1,30 @@
 <?xml version="1.0" ?>
-<robot name="kuka_kr3r540" xmlns:xacro="http://wiki.ros.org/xacro">
+<robot name="kr3r540" xmlns:xacro="http://wiki.ros.org/xacro">
   <xacro:arg name="prefix" default="" />
   <xacro:arg name="use_mock_hardware" default="false" />
+  <xacro:arg name="mock_sensor_commands" default="false" />
+  <xacro:arg name="sim_gazebo_classic" default="false" />
+  <xacro:arg name="sim_gazebo" default="false" />
+  <xacro:arg name="simulation_controllers" default="" />
   <xacro:include filename="$(find kuka_kr3_support)/urdf/kr3r540_macro.xacro"/>
-  <xacro:include filename="$(find kuka_resources)/urdf/common_macro.ros2_control.xacro"/>
-  <xacro:kuka_common_ros2_control_macro name="kr3r540_mock" prefix="$(arg prefix)" use_mock_hardware="$(arg use_mock_hardware)"/>
-  <xacro:kuka_kr3r540 prefix=""/>
+  <!-- <xacro:include filename="$(find kuka_resources)/urdf/common_macro.ros2_control.xacro"/> -->
+  <xacro:include filename="$(find kuka_resources)/urdf/common_sim_macro.ros2_control.xacro"/>
+  <!-- <xacro:kuka_common_ros2_control_macro name="kr3r540_mock" prefix="$(arg prefix)" use_mock_hardware="$(arg use_mock_hardware)"/> -->
+  <!-- <xacro:kr3r540_ros2_control name="kr3r540" prefix="$(arg prefix)" use_mock_hardware="$(arg use_mock_hardware)" simulation_controllers="$(arg simulation_controllers)"/> -->
+   <!-- create link fixed to the "world" -->
+  <link name="world" />
+  <!-- Load robot's macro with parameters -->
+  <!-- set prefix if multiple robots are used -->
+  <xacro:kr3r540 prefix="$(arg prefix)" parent="world" >
+    <origin xyz="0 0 0" rpy="0 0 0" />          <!-- position robot in the world -->
+  </xacro:kr3r540>
+  <xacro:kr3r540_ros2_control
+    name="kr3r540"
+    prefix="$(arg prefix)"
+    use_mock_hardware="$(arg use_mock_hardware)"
+    mock_sensor_commands="$(arg mock_sensor_commands)"
+    sim_gazebo_classic="$(arg sim_gazebo_classic)"
+    sim_gazebo="$(arg sim_gazebo)"
+    simulation_controllers="$(arg simulation_controllers)" />
+  <!-- <xacro:kr3r540 prefix=""/> -->
 </robot>

File: kuka_kr3_support/urdf/kr3r540_macro.xacro (robot description, xacro)
@@ -2,10 +2,11 @@
 <robot xmlns:xacro="http://wiki.ros.org/xacro">
   <xacro:include filename="$(find kuka_resources)/urdf/common_materials.xacro"/>
-  <xacro:macro name="kuka_kr3r540" params="prefix">
+  <xacro:macro name="kr3r540" params="prefix parent *origin">
     <link name="${prefix}base_link">
+      <xacro:default_inertial/>
       <visual>
         <origin xyz="0 0 0" rpy="0 0 0" />
         <geometry>
-          <mesh filename="package://kuka_kr3_support/meshes/kr3r540/visual/base_link.stl" />
+          <mesh filename="file://$(find kuka_kr3_support)/meshes/kr3r540/visual/base_link.stl" />
         </geometry>
         <xacro:material_kuka_pedestal />
@@ -14,13 +15,14 @@
         <origin xyz="0 0 0" rpy="0 0 0" />
         <geometry>
-          <mesh filename="package://kuka_kr3_support/meshes/kr3r540/collision/base_link.stl" />
+          <mesh filename="file://$(find kuka_kr3_support)/meshes/kr3r540/collision/base_link.stl" />
         </geometry>
       </collision>
     </link>
     <link name="${prefix}link_1">
+      <xacro:default_inertial/>
       <visual>
         <origin xyz="0 0 0" rpy="0 0 0" />
         <geometry>
-          <mesh filename="package://kuka_kr3_support/meshes/kr3r540/visual/link_1.stl" />
+          <mesh filename="file://$(find kuka_kr3_support)/meshes/kr3r540/visual/link_1.stl" />
         </geometry>
         <xacro:material_kuka_ral_pure_white />
@@ -29,13 +31,14 @@
         <origin xyz="0 0 0" rpy="0 0 0" />
         <geometry>
-          <mesh filename="package://kuka_kr3_support/meshes/kr3r540/collision/link_1.stl" />
+          <mesh filename="file://$(find kuka_kr3_support)/meshes/kr3r540/collision/link_1.stl" />
         </geometry>
       </collision>
     </link>
     <link name="${prefix}link_2">
+      <xacro:default_inertial/>
       <visual>
         <origin xyz="0 0 0" rpy="0 0 0" />
         <geometry>
-          <mesh filename="package://kuka_kr3_support/meshes/kr3r540/visual/link_2.stl" />
+          <mesh filename="file://$(find kuka_kr3_support)/meshes/kr3r540/visual/link_2.stl" />
         </geometry>
         <xacro:material_kuka_ral_pure_white />
@@ -44,13 +47,14 @@
         <origin xyz="0 0 0" rpy="0 0 0" />
         <geometry>
-          <mesh filename="package://kuka_kr3_support/meshes/kr3r540/collision/link_2.stl" />
+          <mesh filename="file://$(find kuka_kr3_support)/meshes/kr3r540/collision/link_2.stl" />
         </geometry>
       </collision>
     </link>
     <link name="${prefix}link_3">
+      <xacro:default_inertial/>
       <visual>
         <origin xyz="0 0 0" rpy="0 0 0" />
         <geometry>
-          <mesh filename="package://kuka_kr3_support/meshes/kr3r540/visual/link_3.stl" />
+          <mesh filename="file://$(find kuka_kr3_support)/meshes/kr3r540/visual/link_3.stl" />
         </geometry>
         <xacro:material_kuka_ral_pure_white />
@@ -59,13 +63,14 @@
         <origin xyz="0 0 0" rpy="0 0 0" />
         <geometry>
-          <mesh filename="package://kuka_kr3_support/meshes/kr3r540/collision/link_3.stl" />
+          <mesh filename="file://$(find kuka_kr3_support)/meshes/kr3r540/collision/link_3.stl" />
         </geometry>
       </collision>
     </link>
     <link name="${prefix}link_4">
+      <xacro:default_inertial/>
       <visual>
         <origin xyz="0 0 0" rpy="0 0 0" />
         <geometry>
-          <mesh filename="package://kuka_kr3_support/meshes/kr3r540/visual/link_4.stl" />
+          <mesh filename="file://$(find kuka_kr3_support)/meshes/kr3r540/visual/link_4.stl" />
         </geometry>
         <xacro:material_kuka_ral_pure_white />
@@ -74,13 +79,14 @@
         <origin xyz="0 0 0" rpy="0 0 0" />
         <geometry>
-          <mesh filename="package://kuka_kr3_support/meshes/kr3r540/collision/link_4.stl" />
+          <mesh filename="file://$(find kuka_kr3_support)/meshes/kr3r540/collision/link_4.stl" />
         </geometry>
       </collision>
     </link>
     <link name="${prefix}link_5">
+      <xacro:default_inertial/>
       <visual>
         <origin xyz="0 0 0" rpy="0 0 0" />
         <geometry>
-          <mesh filename="package://kuka_kr3_support/meshes/kr3r540/visual/link_5.stl" />
+          <mesh filename="file://$(find kuka_kr3_support)/meshes/kr3r540/visual/link_5.stl" />
         </geometry>
         <xacro:material_kuka_ral_pure_white />
@@ -89,13 +95,14 @@
         <origin xyz="0 0 0" rpy="0 0 0" />
         <geometry>
-          <mesh filename="package://kuka_kr3_support/meshes/kr3r540/collision/link_5.stl" />
+          <mesh filename="file://$(find kuka_kr3_support)/meshes/kr3r540/collision/link_5.stl" />
         </geometry>
       </collision>
     </link>
     <link name="${prefix}link_6">
+      <xacro:default_inertial/>
       <visual>
         <origin xyz="0 0 0" rpy="0 0 0" />
         <geometry>
-          <mesh filename="package://kuka_kr3_support/meshes/kr3r540/visual/link_6.stl" />
+          <mesh filename="file://$(find kuka_kr3_support)/meshes/kr3r540/visual/link_6.stl" />
         </geometry>
         <xacro:material_kuka_pedestal />
@@ -104,5 +111,5 @@
         <origin xyz="0 0 0" rpy="0 0 0" />
         <geometry>
-          <mesh filename="package://kuka_kr3_support/meshes/kr3r540/collision/link_6.stl" />
+          <mesh filename="file://$(find kuka_kr3_support)/meshes/kr3r540/collision/link_6.stl" />
         </geometry>
       </collision>
@@ -110,4 +117,10 @@
     <!-- Following REP199, this frame shall be use to attach EEF or other equipment -->
     <link name="${prefix}flange" />
+    <!-- base_joint fixes base_link to the environment -->
+    <joint name="${prefix}base_joint" type="fixed">
+      <xacro:insert_block name="origin" />
+      <parent link="${parent}" />
+      <child link="${prefix}base_link" />
+    </joint>
     <joint name="${prefix}joint_a1" type="revolute">
       <origin xyz="0 0 0.345" rpy="0 0 0"/>

Commit message: using-external-joints-and-links approach

File: kuka_kr3_support/urdf/kr3r540.xacro (robot description, xacro)
@@ -7,12 +7,17 @@
   <xacro:arg name="sim_gazebo" default="false" />
   <xacro:arg name="simulation_controllers" default="" />
+   <!-- create link fixed to the "world" -->
+   <!-- using-external-joints-and-links approach -->
+  <link name="world" />
+  <joint name="$(arg prefix)base_joint" type="fixed">
+    <origin xyz="0 0 0" rpy="0 0 0" />          <!-- position robot in the world -->
+    <parent link="world" />
+    <child link="$(arg prefix)base_link" />
+  </joint>
   <xacro:include filename="$(find kuka_kr3_support)/urdf/kr3r540_macro.xacro"/>
   <xacro:include filename="$(find kuka_resources)/urdf/common_macro.ros2_control.xacro"/>
-   <!-- create link fixed to the "world" -->
-  <link name="world" />
   <!-- Load robot's macro with parameters -->
   <!-- set prefix if multiple robots are used -->
-  <xacro:kuka_kr3r540 prefix="$(arg prefix)" parent="world" >
-    <origin xyz="0 0 0" rpy="0 0 0" />          <!-- position robot in the world -->
+  <xacro:kuka_kr3r540 prefix="$(arg prefix)" >
   </xacro:kuka_kr3r540>
   <xacro:kuka_common_ros2_control_macro

File: kuka_kr3_support/urdf/kr3r540_macro.xacro (robot description, xacro)
@@ -3,5 +3,5 @@
   <xacro:include filename="$(find kuka_resources)/urdf/common_materials.xacro"/>
   <xacro:include filename="$(find kuka_resources)/urdf/common_properties.xacro"/>
-  <xacro:macro name="kuka_kr3r540" params="prefix parent *origin">
+  <xacro:macro name="kuka_kr3r540" params="prefix">
     <link name="${prefix}base_link">
       <xacro:default_inertial/>
@@ -118,10 +118,4 @@
     <!-- Following REP199, this frame shall be use to attach EEF or other equipment -->
     <link name="${prefix}flange" />
-    <!-- base_joint fixes base_link to the environment -->
-    <joint name="${prefix}base_joint" type="fixed">
-      <xacro:insert_block name="origin" />
-      <parent link="${parent}" />
-      <child link="${prefix}base_link" />
-    </joint>
     <joint name="${prefix}joint_a1" type="revolute">
       <origin xyz="0 0 0.345" rpy="0 0 0"/>
