Commit message: included kuka_lbr to run from common launch file

File: kuka_ros2_control_sim_support/urdf/common_sim_kuka.xacro (robot description, xacro)
@@ -29,4 +29,5 @@
     sim_gazebo="$(arg sim_gazebo)"
     simulation_controllers="$(arg simulation_controllers)"
+    robot_description_package="$(arg robot_description_package)"
     />
   <xacro:if value="${robot_description_package == 'kuka_kr3_support'}">
@@ -75,3 +76,6 @@
     <xacro:kuka_kr210l150 prefix="$(arg prefix)"/>
   </xacro:if>
+  <xacro:if value="${robot_description_package == 'kuka_lbr_iiwa_support'}">
+    <xacro:kuka_lbr_iiwa_14_r820 prefix="$(arg prefix)"/>
+  </xacro:if>
 </robot>

File: kuka_ros2_control_sim_support/urdf/common_sim_macro.ros2_control.xacro (robot description, xacro)
@@ -7,5 +7,6 @@
                sim_gazebo_classic:=^|false
                sim_gazebo:=^|false
-               simulation_controllers"
+               simulation_controllers
+               robot_description_package"
                >
     <ros2_control name="${name}" type="system">
@@ -79,4 +80,15 @@
         </state_interface>
       </joint>
+      <xacro:if value="${robot_description_package == 'kuka_lbr_iiwa_support'}">
+        <joint name="${prefix}joint_a7">
+        <command_interface name="position">
+          <param name="min">-1</param>
+          <param name="max">1</param>
+        </command_interface>
+        <state_interface name="position">
+          <param name="initial_value">0.0</param>
+        </state_interface>
+        </joint>
+      </xacro:if>
     </ros2_control>
     <xacro:if value="$(arg sim_gazebo_classic)">
