Commit message: [URDF] Adding inertial and using `find` for getting package paths for simulators to work (#13)
Co-authored-by: Dr. Denis <denis@stoglrobotics.de>

File: kuka_kr6_support/urdf/kr6r700sixx_macro.xacro (robot description, xacro)
@@ -1,11 +1,14 @@
 <?xml version="1.0"?>
 <robot xmlns:xacro="http://wiki.ros.org/xacro">
+  <xacro:include filename="$(find kuka_resources)/urdf/common_constants.xacro"/>
+  <xacro:include filename="$(find kuka_resources)/urdf/common_properties.xacro"/>
   <xacro:include filename="$(find kuka_resources)/urdf/common_materials.xacro"/>
   <xacro:macro name="kuka_kr6r700sixx" params="prefix">
     <link name="${prefix}base_link">
+      <xacro:default_inertial/>
       <visual>
         <origin xyz="0 0 0" rpy="0 0 0" />
         <geometry>
-          <mesh filename="package://kuka_kr6_support/meshes/kr6_agilus/visual/base_link.dae" />
+          <mesh filename="file://$(find kuka_kr6_support)/meshes/kr6_agilus/visual/base_link.dae" />
         </geometry>
         <xacro:material_kuka_pedestal />
@@ -14,13 +17,14 @@
         <origin xyz="0 0 0" rpy="0 0 0" />
         <geometry>
-          <mesh filename="package://kuka_kr6_support/meshes/kr6_agilus/collision/base_link.stl" />
+          <mesh filename="file://$(find kuka_kr6_support)/meshes/kr6_agilus/collision/base_link.stl" />
         </geometry>
       </collision>
     </link>
     <link name="${prefix}link_1">
+      <xacro:default_inertial/>
       <visual>
         <origin xyz="0 0 0" rpy="0 0 0" />
         <geometry>
-          <mesh filename="package://kuka_kr6_support/meshes/kr6_agilus/visual/link_1.dae" />
+          <mesh filename="file://$(find kuka_kr6_support)/meshes/kr6_agilus/visual/link_1.dae" />
         </geometry>
         <xacro:material_kuka_orange />
@@ -29,13 +33,14 @@
         <origin xyz="0 0 0" rpy="0 0 0" />
         <geometry>
-          <mesh filename="package://kuka_kr6_support/meshes/kr6_agilus/collision/link_1.stl" />
+          <mesh filename="file://$(find kuka_kr6_support)/meshes/kr6_agilus/collision/link_1.stl" />
         </geometry>
       </collision>
     </link>
     <link name="${prefix}link_2">
+      <xacro:default_inertial/>
       <visual>
         <origin xyz="0 0 0" rpy="0 0 0" />
         <geometry>
-          <mesh filename="package://kuka_kr6_support/meshes/kr6r700sixx/visual/link_2.dae" />
+          <mesh filename="file://$(find kuka_kr6_support)/meshes/kr6r700sixx/visual/link_2.dae" />
         </geometry>
         <xacro:material_kuka_orange />
@@ -44,13 +49,14 @@
         <origin xyz="0 0 0" rpy="0 0 0" />
         <geometry>
-          <mesh filename="package://kuka_kr6_support/meshes/kr6r700sixx/collision/link_2.stl" />
+          <mesh filename="file://$(find kuka_kr6_support)/meshes/kr6r700sixx/collision/link_2.stl" />
         </geometry>
       </collision>
     </link>
     <link name="${prefix}link_3">
+      <xacro:default_inertial/>
       <visual>
         <origin xyz="0 0 0" rpy="0 0 0" />
         <geometry>
-          <mesh filename="package://kuka_kr6_support/meshes/kr6_agilus/visual/link_3.dae" />
+          <mesh filename="file://$(find kuka_kr6_support)/meshes/kr6_agilus/visual/link_3.dae" />
         </geometry>
         <xacro:material_kuka_orange />
@@ -59,13 +65,14 @@
         <origin xyz="0 0 0" rpy="0 0 0" />
         <geometry>
-          <mesh filename="package://kuka_kr6_support/meshes/kr6_agilus/collision/link_3.stl" />
+          <mesh filename="file://$(find kuka_kr6_support)/meshes/kr6_agilus/collision/link_3.stl" />
         </geometry>
       </collision>
     </link>
     <link name="${prefix}link_4">
+      <xacro:default_inertial/>
       <visual>
         <origin xyz="0 0 0" rpy="0 0 0" />
         <geometry>
-          <mesh filename="package://kuka_kr6_support/meshes/kr6r700sixx/visual/link_4.dae" />
+          <mesh filename="file://$(find kuka_kr6_support)/meshes/kr6r700sixx/visual/link_4.dae" />
         </geometry>
         <xacro:material_kuka_orange />
@@ -74,13 +81,14 @@
         <origin xyz="0 0 0" rpy="0 0 0" />
         <geometry>
-          <mesh filename="package://kuka_kr6_support/meshes/kr6r700sixx/collision/link_4.stl" />
+          <mesh filename="file://$(find kuka_kr6_support)/meshes/kr6r700sixx/collision/link_4.stl" />
         </geometry>
       </collision>
     </link>
     <link name="${prefix}link_5">
+      <xacro:default_inertial/>
       <visual>
         <origin xyz="0 0 0" rpy="0 0 0" />
         <geometry>
-          <mesh filename="package://kuka_kr6_support/meshes/kr6_agilus/visual/link_5.dae" />
+          <mesh filename="file://$(find kuka_kr6_support)/meshes/kr6_agilus/visual/link_5.dae" />
         </geometry>
         <xacro:material_kuka_orange />
@@ -89,13 +97,14 @@
         <origin xyz="0 0 0" rpy="0 0 0" />
         <geometry>
-          <mesh filename="package://kuka_kr6_support/meshes/kr6_agilus/collision/link_5.stl" />
+          <mesh filename="file://$(find kuka_kr6_support)/meshes/kr6_agilus/collision/link_5.stl" />
         </geometry>
       </collision>
     </link>
     <link name="${prefix}link_6">
+      <xacro:default_inertial/>
       <visual>
         <origin xyz="0 0 0" rpy="0 0 0" />
         <geometry>
-          <mesh filename="package://kuka_kr6_support/meshes/kr6_agilus/visual/link_6.dae" />
+          <mesh filename="file://$(find kuka_kr6_support)/meshes/kr6_agilus/visual/link_6.dae" />
         </geometry>
         <xacro:material_kuka_pedestal />
@@ -104,5 +113,5 @@
         <origin xyz="0 0 0" rpy="0 0 0" />
         <geometry>
-          <mesh filename="package://kuka_kr6_support/meshes/kr6_agilus/collision/link_6.stl" />
+          <mesh filename="file://$(find kuka_kr6_support)/meshes/kr6_agilus/collision/link_6.stl" />
         </geometry>
       </collision>

File: kuka_kr6_support/urdf/kr6r900sixx_macro.xacro (robot description, xacro)
@@ -2,10 +2,12 @@
 <robot xmlns:xacro="http://wiki.ros.org/xacro">
   <xacro:include filename="$(find kuka_resources)/urdf/common_materials.xacro"/>
+  <xacro:include filename="$(find kuka_resources)/urdf/common_properties.xacro"/>
   <xacro:macro name="kuka_kr6r900sixx" params="prefix">
     <link name="${prefix}base_link">
+      <xacro:default_inertial/>
       <visual>
         <origin xyz="0 0 0" rpy="0 0 0"/>
         <geometry>
-          <mesh filename="package://kuka_kr6_support/meshes/kr6_agilus/visual/base_link.dae" />
+          <mesh filename="file://$(find kuka_kr6_support)/meshes/kr6_agilus/visual/base_link.dae" />
         </geometry>
         <xacro:material_kuka_pedestal />
@@ -14,13 +16,14 @@
         <origin xyz="0 0 0" rpy="0 0 0"/>
         <geometry>
-          <mesh filename="package://kuka_kr6_support/meshes/kr6_agilus/collision/base_link.stl" />
+          <mesh filename="file://$(find kuka_kr6_support)/meshes/kr6_agilus/collision/base_link.stl" />
         </geometry>
       </collision>
     </link>
     <link name="${prefix}link_1">
+      <xacro:default_inertial/>
       <visual>
         <origin xyz="0 0 0" rpy="0 0 0"/>
         <geometry>
-          <mesh filename="package://kuka_kr6_support/meshes/kr6_agilus/visual/link_1.dae" />
+          <mesh filename="file://$(find kuka_kr6_support)/meshes/kr6_agilus/visual/link_1.dae" />
         </geometry>
         <xacro:material_kuka_orange />
@@ -29,13 +32,14 @@
         <origin xyz="0 0 0" rpy="0 0 0"/>
         <geometry>
-          <mesh filename="package://kuka_kr6_support/meshes/kr6_agilus/collision/link_1.stl" />
+          <mesh filename="file://$(find kuka_kr6_support)/meshes/kr6_agilus/collision/link_1.stl" />
         </geometry>
       </collision>
     </link>
     <link name="${prefix}link_2">
+      <xacro:default_inertial/>
       <visual>
         <origin xyz="0 0 0" rpy="0 0 0"/>
         <geometry>
-          <mesh filename="package://kuka_kr6_support/meshes/kr6r900sixx/visual/link_2.dae"/>
+          <mesh filename="file://$(find kuka_kr6_support)/meshes/kr6r900sixx/visual/link_2.dae"/>
         </geometry>
         <xacro:material_kuka_orange />
@@ -44,13 +48,14 @@
         <origin xyz="0 0 0" rpy="0 0 0"/>
         <geometry>
-          <mesh filename="package://kuka_kr6_support/meshes/kr6r900sixx/collision/link_2.stl" />
+          <mesh filename="file://$(find kuka_kr6_support)/meshes/kr6r900sixx/collision/link_2.stl" />
         </geometry>
       </collision>
     </link>
     <link name="${prefix}link_3">
+      <xacro:default_inertial/>
       <visual>
         <origin xyz="0 0 0" rpy="0 0 0"/>
         <geometry>
-          <mesh filename="package://kuka_kr6_support/meshes/kr6_agilus/visual/link_3.dae" />
+          <mesh filename="file://$(find kuka_kr6_support)/meshes/kr6_agilus/visual/link_3.dae" />
         </geometry>
         <xacro:material_kuka_orange />
@@ -59,13 +64,14 @@
         <origin xyz="0 0 0" rpy="0 0 0"/>
         <geometry>
-          <mesh filename="package://kuka_kr6_support/meshes/kr6_agilus/collision/link_3.stl" />
+          <mesh filename="file://$(find kuka_kr6_support)/meshes/kr6_agilus/collision/link_3.stl" />
         </geometry>
       </collision>
     </link>
     <link name="${prefix}link_4">
+      <xacro:default_inertial/>
       <visual>
         <origin xyz="0 0 0" rpy="0 0 0"/>
         <geometry>
-          <mesh filename="package://kuka_kr6_support/meshes/kr6r900sixx/visual/link_4.dae" />
+          <mesh filename="file://$(find kuka_kr6_support)/meshes/kr6r900sixx/visual/link_4.dae" />
         </geometry>
         <xacro:material_kuka_orange />
@@ -74,13 +80,14 @@
         <origin xyz="0 0 0" rpy="0 0 0"/>
         <geometry>
-          <mesh filename="package://kuka_kr6_support/meshes/kr6r900sixx/collision/link_4.stl" />
+          <mesh filename="file://$(find kuka_kr6_support)/meshes/kr6r900sixx/collision/link_4.stl" />
         </geometry>
       </collision>
     </link>
     <link name="${prefix}link_5">
+      <xacro:default_inertial/>
       <visual>
         <origin xyz="0 0 0" rpy="0 0 0"/>
         <geometry>
-          <mesh filename="package://kuka_kr6_support/meshes/kr6_agilus/visual/link_5.dae" />
+          <mesh filename="file://$(find kuka_kr6_support)/meshes/kr6_agilus/visual/link_5.dae" />
         </geometry>
         <xacro:material_kuka_orange />
@@ -89,13 +96,14 @@
         <origin xyz="0 0 0" rpy="0 0 0"/>
         <geometry>
-          <mesh filename="package://kuka_kr6_support/meshes/kr6_agilus/collision/link_5.stl" />
+          <mesh filename="file://$(find kuka_kr6_support)/meshes/kr6_agilus/collision/link_5.stl" />
         </geometry>
       </collision>
     </link>
     <link name="${prefix}link_6">
+      <xacro:default_inertial/>
       <visual>
         <origin xyz="0 0 0" rpy="0 0 0"/>
         <geometry>
-          <mesh filename="package://kuka_kr6_support/meshes/kr6_agilus/visual/link_6.dae" />
+          <mesh filename="file://$(find kuka_kr6_support)/meshes/kr6_agilus/visual/link_6.dae" />
         </geometry>
         <xacro:material_kuka_pedestal />
@@ -104,5 +112,5 @@
         <origin xyz="0 0 0" rpy="0 0 0"/>
         <geometry>
-          <mesh filename="package://kuka_kr6_support/meshes/kr6_agilus/collision/link_6.stl" />
+          <mesh filename="file://$(find kuka_kr6_support)/meshes/kr6_agilus/collision/link_6.stl" />
         </geometry>
       </collision>

File: kuka_lbr_iiwa_support/urdf/lbr_iiwa_14_r820_macro.xacro (robot description, xacro)
@@ -2,10 +2,12 @@
 <robot xmlns:xacro="http://wiki.ros.org/xacro">
   <xacro:macro name="kuka_lbr_iiwa_14_r820" params="prefix">
+  <xacro:include filename="$(find kuka_resources)/urdf/common_properties.xacro"/>
     <!-- link list -->
     <link name="${prefix}base_link">
+      <xacro:default_inertial/>
       <visual>
         <origin xyz="0 0 0" rpy="0 0 0" />
         <geometry>
-          <mesh filename="package://kuka_lbr_iiwa_support/meshes/lbr_iiwa_14_r820/visual/base_link.dae" />
+          <mesh filename="file://$(find kuka_lbr_iiwa_support)/meshes/lbr_iiwa_14_r820/visual/base_link.dae" />
         </geometry>
       </visual>
@@ -13,13 +15,14 @@
         <origin xyz="0 0 0" rpy="0 0 0" />
         <geometry>
-          <mesh filename="package://kuka_lbr_iiwa_support/meshes/lbr_iiwa_14_r820/collision/base_link.stl" />
+          <mesh filename="file://$(find kuka_lbr_iiwa_support)/meshes/lbr_iiwa_14_r820/collision/base_link.stl" />
         </geometry>
       </collision>
     </link>
     <link name="${prefix}link_1">
+      <xacro:default_inertial/>
       <visual>
         <origin xyz="0 0 0" rpy="0 0 0" />
         <geometry>
-          <mesh filename="package://kuka_lbr_iiwa_support/meshes/lbr_iiwa_14_r820/visual/link_1.dae" />
+          <mesh filename="file://$(find kuka_lbr_iiwa_support)/meshes/lbr_iiwa_14_r820/visual/link_1.dae" />
         </geometry>
       </visual>
@@ -27,13 +30,14 @@
         <origin xyz="0 0 0" rpy="0 0 0" />
         <geometry>
-          <mesh filename="package://kuka_lbr_iiwa_support/meshes/lbr_iiwa_14_r820/collision/link_1.stl" />
+          <mesh filename="file://$(find kuka_lbr_iiwa_support)/meshes/lbr_iiwa_14_r820/collision/link_1.stl" />
         </geometry>
       </collision>
     </link>
     <link name="${prefix}link_2">
+      <xacro:default_inertial/>
       <visual>
         <origin xyz="0 0 0" rpy="0 0 0" />
         <geometry>
-          <mesh filename="package://kuka_lbr_iiwa_support/meshes/lbr_iiwa_14_r820/visual/link_2.dae" />
+          <mesh filename="file://$(find kuka_lbr_iiwa_support)/meshes/lbr_iiwa_14_r820/visual/link_2.dae" />
         </geometry>
       </visual>
@@ -41,13 +45,14 @@
         <origin xyz="0 0 0" rpy="0 0 0" />
         <geometry>
-          <mesh filename="package://kuka_lbr_iiwa_support/meshes/lbr_iiwa_14_r820/collision/link_2.stl" />
+          <mesh filename="file://$(find kuka_lbr_iiwa_support)/meshes/lbr_iiwa_14_r820/collision/link_2.stl" />
         </geometry>
       </collision>
     </link>
     <link name="${prefix}link_3">
+      <xacro:default_inertial/>
       <visual>
         <origin xyz="0 0 0" rpy="0 0 0" />
         <geometry>
-          <mesh filename="package://kuka_lbr_iiwa_support/meshes/lbr_iiwa_14_r820/visual/link_3.dae" />
+          <mesh filename="file://$(find kuka_lbr_iiwa_support)/meshes/lbr_iiwa_14_r820/visual/link_3.dae" />
         </geometry>
       </visual>
@@ -55,13 +60,14 @@
         <origin xyz="0 0 0" rpy="0 0 0" />
         <geometry>
-          <mesh filename="package://kuka_lbr_iiwa_support/meshes/lbr_iiwa_14_r820/collision/link_3.stl" />
+          <mesh filename="file://$(find kuka_lbr_iiwa_support)/meshes/lbr_iiwa_14_r820/collision/link_3.stl" />
         </geometry>
       </collision>
     </link>
     <link name="${prefix}link_4">
+      <xacro:default_inertial/>
       <visual>
         <origin xyz="0 0 0" rpy="0 0 0" />
         <geometry>
-          <mesh filename="package://kuka_lbr_iiwa_support/meshes/lbr_iiwa_14_r820/visual/link_4.dae" />
+          <mesh filename="file://$(find kuka_lbr_iiwa_support)/meshes/lbr_iiwa_14_r820/visual/link_4.dae" />
         </geometry>
       </visual>
@@ -69,13 +75,14 @@
         <origin xyz="0 0 0" rpy="0 0 0" />
         <geometry>
-          <mesh filename="package://kuka_lbr_iiwa_support/meshes/lbr_iiwa_14_r820/collision/link_4.stl" />
+          <mesh filename="file://$(find kuka_lbr_iiwa_support)/meshes/lbr_iiwa_14_r820/collision/link_4.stl" />
         </geometry>
       </collision>
     </link>
     <link name="${prefix}link_5">
+      <xacro:default_inertial/>
       <visual>
         <origin xyz="0 0 0" rpy="0 0 0" />
         <geometry>
-          <mesh filename="package://kuka_lbr_iiwa_support/meshes/lbr_iiwa_14_r820/visual/link_5.dae" />
+          <mesh filename="file://$(find kuka_lbr_iiwa_support)/meshes/lbr_iiwa_14_r820/visual/link_5.dae" />
         </geometry>
       </visual>
@@ -83,13 +90,14 @@
         <origin xyz="0 0 0" rpy="0 0 0" />
         <geometry>
-          <mesh filename="package://kuka_lbr_iiwa_support/meshes/lbr_iiwa_14_r820/collision/link_5.stl" />
+          <mesh filename="file://$(find kuka_lbr_iiwa_support)/meshes/lbr_iiwa_14_r820/collision/link_5.stl" />
         </geometry>
       </collision>
     </link>
     <link name="${prefix}link_6">
+      <xacro:default_inertial/>
       <visual>
         <origin xyz="0 0 0" rpy="0 0 0" />
         <geometry>
-          <mesh filename="package://kuka_lbr_iiwa_support/meshes/lbr_iiwa_14_r820/visual/link_6.dae" />
+          <mesh filename="file://$(find kuka_lbr_iiwa_support)/meshes/lbr_iiwa_14_r820/visual/link_6.dae" />
         </geometry>
       </visual>
@@ -97,13 +105,14 @@
         <origin xyz="0 0 0" rpy="0 0 0" />
         <geometry>
-          <mesh filename="package://kuka_lbr_iiwa_support/meshes/lbr_iiwa_14_r820/collision/link_6.stl" />
+          <mesh filename="file://$(find kuka_lbr_iiwa_support)/meshes/lbr_iiwa_14_r820/collision/link_6.stl" />
         </geometry>
       </collision>
     </link>
     <link name="${prefix}link_7">
+      <xacro:default_inertial/>
       <visual>
         <origin xyz="0 0 0" rpy="0 0 0" />
         <geometry>
-          <mesh filename="package://kuka_lbr_iiwa_support/meshes/lbr_iiwa_14_r820/visual/link_7.dae" />
+          <mesh filename="file://$(find kuka_lbr_iiwa_support)/meshes/lbr_iiwa_14_r820/visual/link_7.dae" />
         </geometry>
       </visual>
@@ -111,5 +120,5 @@
         <origin xyz="0 0 0" rpy="0 0 0" />
         <geometry>
-          <mesh filename="package://kuka_lbr_iiwa_support/meshes/lbr_iiwa_14_r820/collision/link_7.stl" />
+          <mesh filename="file://$(find kuka_lbr_iiwa_support)/meshes/lbr_iiwa_14_r820/collision/link_7.stl" />
         </geometry>
       </collision>
