Commit message: move plugin to rsi and extract control stuff

File: common_6dof_position_only_system/control/kuka_6dof_system_position_only.ros2_control.xacro (robot description, xacro)
@@ -1,10 +1,16 @@
 <?xml version="1.0"?>
 <robot xmlns:xacro="http://www.ros.org/wiki/xacro">
-  <xacro:macro name="robot6dof_system_position_only" params="name prefix">
+  <xacro:macro name="kuka_6dof_system_posiition_only" params="name prefix use_mock_hw:=^|false use_mock_sensor_commands:=^|false">
     <ros2_control name="${name}" type="system">
       <hardware>
-        <plugin>ros2_control_kuka_driver/KukaSystemPositionOnlyHardware</plugin>
-        <param name="listen_address">127.0.0.1</param>
-        <param name="listen_port">49152</param>
+        <xacro:if value="${use_mock_hw}">
+          <plugin>mock_components/GenericSystem</plugin>
+          <param name="mock_sensor_commands">${use_mock_sensor_commands}</param>
+        </xacro:if>
+        <xacro:unless value="${use_mock_hw}">
+          <plugin>kuka_rsi_hw_interface/KukaSystemPositionOnlyHardware</plugin>
+          <param name="listen_address">127.0.0.1</param>
+          <param name="listen_port">49152</param>
+        </xacro:unless>
       </hardware>
       <joint name="${prefix}joint_a1">
@@ -13,5 +19,7 @@
           <param name="max">1</param>
         </command_interface>
-        <state_interface name="position"/>
+        <state_interface name="position">
+          <param name="initial_value">0.0</param>
+        </state_interface>
       </joint>
       <joint name="${prefix}joint_a2">
@@ -20,12 +28,16 @@
           <param name="max">1</param>
         </command_interface>
-        <state_interface name="position"/>
+        <state_interface name="position">
+          <param name="initial_value">0.0</param>
+        </state_interface>
 	  </joint>
       <joint name="${prefix}joint_a3">
         <command_interface name="position">
           <param name="min">-1</param>
-          <param name="max">1</param>
+          <param name="max">0.61</param>
         </command_interface>
-        <state_interface name="position"/>
+        <state_interface name="position">
+          <param name="initial_value">0.0</param>
+        </state_interface>
 	  </joint>
       <joint name="${prefix}joint_a4">
@@ -34,5 +46,7 @@
           <param name="max">1</param>
         </command_interface>
-        <state_interface name="position"/>
+        <state_interface name="position">
+          <param name="initial_value">0.0</param>
+        </state_interface>
       </joint>
       <joint name="${prefix}joint_a5">
@@ -41,5 +55,7 @@
           <param name="max">1</param>
         </command_interface>
-        <state_interface name="position"/>
+        <state_interface name="position">
+          <param name="initial_value">0.0</param>
+        </state_interface>
       </joint>
       <joint name="${prefix}joint_a6">
@@ -48,5 +64,7 @@
           <param name="max">1</param>
         </command_interface>
-        <state_interface name="position"/>
+        <state_interface name="position">
+          <param name="initial_value">0.0</param>
+        </state_interface>
       </joint>
     </ros2_control>

File: kuka_kr16_support/urdf/kr16_2.urdf.xacro (robot description, xacro)
@@ -5,6 +5,6 @@
   <xacro:arg name="use_mock_sensor_commands" default="false" />
   <xacro:include filename="$(find kuka_kr16_support)/urdf/kr16_2_macro.xacro" />
-  <xacro:include filename="$(find ros2_control_kuka_driver)/description/kuka_kr16/controllers/kuka_kr16_2_6dof_system.ros2_control.xacro"/>
+  <xacro:include filename="$(find common_6dof_position_only_system)/control/kuka_6dof_system_position_only.ros2_control.xacro"/>
   <xacro:kuka_kr16_2 prefix=""/>
-  <xacro:kuka_kr_16_2_6dof_system name="kuka_kr16_2_mock" prefix="$(arg prefix)" use_mock_hw="$(arg use_mock_hw)" use_mock_sensor_commands="$(arg use_mock_sensor_commands)"/>
+  <xacro:kuka_6dof_system_posiition_only name="kuka_kr16_2_mock" prefix="$(arg prefix)" use_mock_hw="$(arg use_mock_hw)" use_mock_sensor_commands="$(arg use_mock_sensor_commands)"/>
 </robot>

Commit message: add some options for startup of kuka_kr16_bringup

File: common_6dof_position_only_system/control/kuka_6dof_system_position_only.ros2_control.xacro (robot description, xacro)
@@ -1,5 +1,5 @@
 <?xml version="1.0"?>
 <robot xmlns:xacro="http://www.ros.org/wiki/xacro">
-  <xacro:macro name="kuka_6dof_system_posiition_only" params="name prefix use_mock_hw:=^|false use_mock_sensor_commands:=^|false">
+  <xacro:macro name="kuka_6dof_system_posiition_only" params="name prefix use_mock_hw:=^|false use_mock_sensor_commands:=^|false listen_ip_address:=^|127.0.0.1 listen_port:=^|49152">
     <ros2_control name="${name}" type="system">
       <hardware>
@@ -10,6 +10,6 @@
         <xacro:unless value="${use_mock_hw}">
           <plugin>kuka_rsi_hw_interface/KukaSystemPositionOnlyHardware</plugin>
-          <param name="listen_address">172.20.19.101</param>
-          <param name="listen_port">49152</param>
+          <param name="listen_address">${listen_ip_address}</param>
+          <param name="listen_port">${listen_port}</param>
         </xacro:unless>
       </hardware>

File: kuka_kr16_support/urdf/kr16_2.urdf.xacro (robot description, xacro)
@@ -4,7 +4,9 @@
   <xacro:arg name="use_mock_hw" default="false" />
   <xacro:arg name="use_mock_sensor_commands" default="false" />
+  <xacro:arg name="listen_ip_address" default="127.0.0.1" />
+  <xacro:arg name="listen_port" default="49152" />
   <xacro:include filename="$(find kuka_kr16_support)/urdf/kr16_2_macro.xacro" />
   <xacro:include filename="$(find common_6dof_position_only_system)/control/kuka_6dof_system_position_only.ros2_control.xacro"/>
   <xacro:kuka_kr16_2 prefix=""/>
-  <xacro:kuka_6dof_system_posiition_only name="kuka_kr16_2_mock" prefix="$(arg prefix)" use_mock_hw="$(arg use_mock_hw)" use_mock_sensor_commands="$(arg use_mock_sensor_commands)"/>
+  <xacro:kuka_6dof_system_posiition_only name="kuka_kr16_2_mock" prefix="$(arg prefix)" use_mock_hw="$(arg use_mock_hw)" use_mock_sensor_commands="$(arg use_mock_sensor_commands)" listen_ip_address="$(arg listen_ip_address)" listen_port="$(arg listen_port)"/>
 </robot>
