Commit message: functional ros2_control support for kuka base models

File: kuka_ros2_control_support/urdf/common_kuka.xacro (robot description, xacro)
@@ -1,10 +1,12 @@
 <?xml version="1.0" ?>
-<robot name="kuka_kr3r540" xmlns:xacro="http://wiki.ros.org/xacro">
+<robot name="kuka" xmlns:xacro="http://wiki.ros.org/xacro">
   <xacro:arg name="prefix" default="" />
   <xacro:arg name="use_mock_hardware" default="false" />
-  <xacro:arg name="mock_sensor_commands" default="false" />
-  <xacro:arg name="sim_gazebo_classic" default="false" />
-  <xacro:arg name="sim_gazebo" default="false" />
-  <xacro:arg name="simulation_controllers" default="" />
+  <xacro:arg name="robot_description_package" default="kuka_kr3_support"/>
+  <xacro:arg name="robot_description_macro_file" default="kr3r540_macro.xacro"/>
+  <xacro:arg name="robot_name" default="kuka_kr3r540"/>
+  <xacro:property name="robot_description_package" value="$(arg robot_description_package)"/>
+  <xacro:property name="robot_description_macro_file" value="$(arg robot_description_macro_file)"/>
+  <xacro:property name="robot_name" value="$(arg robot_name)"/>
    <!-- create link fixed to the "world" -->
    <!-- using-external-joints-and-links approach -->
@@ -13,19 +15,57 @@
     <origin xyz="0 0 0" rpy="0 0 0" />          <!-- position robot in the world -->
     <parent link="world" />
-    <child link="$(arg prefix)base_link" />
+    <child link="$(arg prefix)base_link"/>
   </joint>
-  <xacro:include filename="$(find kuka_kr3_support)/urdf/kr3r540_macro.xacro"/>
-  <xacro:include filename="$(find kuka_resources)/urdf/common_macro.ros2_control.xacro"/>
-  <!-- Load robot's macro with parameters -->
-  <!-- set prefix if multiple robots are used -->
-  <xacro:kuka_kr3r540 prefix="$(arg prefix)" >
-  </xacro:kuka_kr3r540>
+  <xacro:include filename="$(find ${robot_description_package})/urdf/${robot_description_macro_file}"/>
+  <xacro:include filename="$(find kuka_ros2_control_support)/urdf/common_macro.ros2_control.xacro"/>
   <xacro:kuka_common_ros2_control_macro
-    name="kuka_kr3r540"
+    name="$(arg robot_name)"
     prefix="$(arg prefix)"
     use_mock_hardware="$(arg use_mock_hardware)"
-    mock_sensor_commands="$(arg mock_sensor_commands)"
-    sim_gazebo_classic="$(arg sim_gazebo_classic)"
-    sim_gazebo="$(arg sim_gazebo)"
-    simulation_controllers="$(arg simulation_controllers)" />
+    />
+  <xacro:if value="${robot_description_package == 'kuka_kr3_support'}">
+    <xacro:kuka_kr3r540 prefix="$(arg prefix)"/>
+  </xacro:if>
+  <xacro:if value="${robot_description_package == 'kuka_kr5_support'}">
+    <xacro:kuka_kr5_arc prefix="$(arg prefix)"/>
+  </xacro:if>
+  <xacro:if value="${robot_description_package == 'kuka_kr6_support'}">
+    <xacro:if value="${robot_description_macro_file == 'kr6r700sixx_macro.xacro'}">
+      <xacro:kuka_kr6r700sixx prefix="$(arg prefix)"/>
+    </xacro:if>
+    <xacro:if value="${robot_description_macro_file == 'kr6r900_2_macro.xacro'}">
+      <xacro:kuka_kr6r900_2 prefix="$(arg prefix)"/>
+    </xacro:if>
+    <xacro:if value="${robot_description_macro_file == 'kr6r900sixx_macro.xacro'}">
+      <xacro:kuka_kr6r900sixx prefix="$(arg prefix)"/>
+    </xacro:if>
+  </xacro:if>
+  <xacro:if value="${robot_description_package == 'kuka_kr10_support'}">
+    <xacro:if value="${robot_description_macro_file == 'kr10r900_2_macro.xacro'}">
+      <xacro:kuka_kr10r900_2 prefix="$(arg prefix)"/>
+    </xacro:if>
+    <xacro:if value="${robot_description_macro_file == 'kr10r1100sixx_macro.xacro'}">
+      <xacro:kuka_kr10r1100sixx prefix="$(arg prefix)"/>
+    </xacro:if>
+    <xacro:if value="${robot_description_macro_file == 'kr10r1420_macro.xacro'}">
+      <xacro:kuka_kr10r1420 prefix="$(arg prefix)"/>
+    </xacro:if>
+  </xacro:if>
+  <xacro:if value="${robot_description_package == 'kuka_kr16_support'}">
+    <xacro:kuka_kr16_2 prefix="$(arg prefix)"/>
+  </xacro:if>
+  <xacro:if value="${robot_description_package == 'kuka_kr120_support'}">
+    <xacro:kuka_kr120r2500pro prefix="$(arg prefix)"/>
+  </xacro:if>
+  <xacro:if value="${robot_description_package == 'kuka_kr150_support'}">
+    <xacro:if value="${robot_description_macro_file == 'kr150_2_macro.xacro'}">
+      <xacro:kuka_kr150_2 prefix="$(arg prefix)"/>
+    </xacro:if>
+    <xacro:if value="${robot_description_macro_file == 'kr150r3100_2_macro.xacro'}">
+      <xacro:kuka_kr150r3100_2 prefix="$(arg prefix)"/>
+    </xacro:if>
+  </xacro:if>
+  <xacro:if value="${robot_description_package == 'kuka_kr210_support'}">
+    <xacro:kuka_kr210l150 prefix="$(arg prefix)"/>
+  </xacro:if>
 </robot>

File: kuka_ros2_control_support/urdf/common_macro.ros2_control.xacro (robot description, xacro)
@@ -4,25 +4,10 @@
                name
                prefix
-               use_mock_hardware:=^|false
-               mock_sensor_commands:=^|false
-               sim_gazebo_classic:=^|false
-               sim_gazebo:=^|false
-               simulation_controllers"
-               >
+               use_mock_hardware:=^|false">
     <ros2_control name="${name}" type="system">
       <hardware>
         <xacro:if value="${use_mock_hardware}">
           <plugin>mock_components/GenericSystem</plugin>
-          <param name="mock_sensor_commands">${mock_sensor_commands}</param>
         </xacro:if>
-        <xacro:if value="${sim_gazebo_classic}">
-          <plugin>gazebo_ros2_control/GazeboSystem</plugin>
-        </xacro:if>
-        <xacro:if value="${sim_gazebo}">
-          <plugin>ign_ros2_control/IgnitionSystem</plugin>
-        </xacro:if>
-        <xacro:unless value="${use_mock_hardware or sim_gazebo_classic or sim_gazebo}">
-          <plugin>robot_hardware_inteface/RobotHardwareInteface</plugin>
-        </xacro:unless>
       </hardware>
       <joint name="${prefix}joint_a1">
@@ -80,47 +65,5 @@
         </state_interface>
       </joint>
-      <sensor name="tcp_fts_sensor">            <!-- Remove/change sensors as needed -->
-        <state_interface name="fx"/>
-        <state_interface name="fy"/>
-        <state_interface name="fz"/>
-        <state_interface name="tx"/>
-        <state_interface name="ty"/>
-        <state_interface name="tz"/>
-        <param name="frame_id">tool0</param>    <!-- Change sensors as needed -->
-        <param name="min_fx">-100</param>
-        <param name="max_fx">100</param>
-        <param name="min_fy">-100</param>
-        <param name="max_fy">100</param>
-        <param name="min_fz">-200</param>
-        <param name="max_fz">200</param>
-        <param name="min_tx">-10</param>
-        <param name="max_tx">10</param>
-        <param name="min_ty">-10</param>
-        <param name="max_ty">10</param>
-        <param name="min_tz">-15</param>
-        <param name="max_tz">15</param>
-      </sensor>
     </ros2_control>
-    <xacro:if value="$(arg sim_gazebo_classic)">
-      <!-- Gazebo plugins -->
-      <gazebo reference="world">
-      </gazebo>
-      <gazebo>
-        <plugin filename="libgazebo_ros2_control.so" name="gazebo_ros2_control">
-          <parameters>${simulation_controllers}</parameters>
-        </plugin>
-      </gazebo>
-    </xacro:if>
-    <xacro:if value="$(arg sim_gazebo)">
-      <!-- Gazebo plugins -->
-      <gazebo reference="world">
-      </gazebo>
-      <gazebo>
-        <plugin filename="libign_ros2_control-system.so" name="ign_ros2_control::IgnitionROS2ControlPlugin">
-          <parameters>${simulation_controllers}</parameters>
-          <controller_manager_node_name>${prefix}controller_manager</controller_manager_node_name>
-        </plugin>
-      </gazebo>
-    </xacro:if>
   </xacro:macro>
 </robot>

Commit message: included kuka_lbr in the comman launch and xacro files

File: kuka_ros2_control_support/urdf/common_kuka.xacro (robot description, xacro)
@@ -3,7 +3,7 @@
   <xacro:arg name="prefix" default="" />
   <xacro:arg name="use_mock_hardware" default="false" />
-  <xacro:arg name="robot_description_package"/>
-  <xacro:arg name="robot_description_macro_file"/>
-  <xacro:arg name="robot_name"/>
+  <xacro:arg name="robot_description_package" default="kuka_kr3_support"/>
+  <xacro:arg name="robot_description_macro_file" default="kr3r540_macro.xacro"/>
+  <xacro:arg name="robot_name" default="kuka_kr3r540"/>
   <xacro:property name="robot_description_package" value="$(arg robot_description_package)"/>
   <xacro:property name="robot_description_macro_file" value="$(arg robot_description_macro_file)"/>
@@ -23,4 +23,5 @@
     prefix="$(arg prefix)"
     use_mock_hardware="$(arg use_mock_hardware)"
+    robot_description_package="$(arg robot_description_package)"
     />
   <xacro:if value="${robot_description_package == 'kuka_kr3_support'}">
@@ -69,3 +70,6 @@
     <xacro:kuka_kr210l150 prefix="$(arg prefix)"/>
   </xacro:if>
+  <xacro:if value="${robot_description_package == 'kuka_lbr_iiwa_support'}">
+    <xacro:kuka_lbr_iiwa_14_r820 prefix="$(arg prefix)"/>
+  </xacro:if>
 </robot>

File: kuka_ros2_control_support/urdf/common_macro.ros2_control.xacro (robot description, xacro)
@@ -4,5 +4,7 @@
                name
                prefix
-               use_mock_hardware:=^|false">
+               use_mock_hardware:=^|false
+               robot_description_package"
+               >
     <ros2_control name="${name}" type="system">
       <hardware>
@@ -65,4 +67,15 @@
         </state_interface>
       </joint>
+      <xacro:if value="${robot_description_package == 'kuka_lbr_iiwa_support'}">
+        <joint name="${prefix}joint_a7">
+        <command_interface name="position">
+          <param name="min">-1</param>
+          <param name="max">1</param>
+        </command_interface>
+        <state_interface name="position">
+          <param name="initial_value">0.0</param>
+        </state_interface>
+        </joint>
+      </xacro:if>
     </ros2_control>
   </xacro:macro>

Commit message: removed inital_positions arg not needed as initial_valu specified in stateinterface

File: kuka_ros2_control_support/urdf/common_kuka.xacro (robot description, xacro)
@@ -9,5 +9,4 @@
   <xacro:arg name="robot_description_macro_file" default="kr3r540_macro.xacro"/>
   <xacro:arg name="robot_name" default="kuka_kr3r540"/>
-  <xacro:arg name="initial_positions_file" default="$(find kuka_ros2_control_support)/config/initial_positions.yaml"/>
   <xacro:arg name="robot_ip" default="10.181.116.41"/>
   <xacro:arg name="robot_port" default="54600"/>
@@ -33,5 +32,4 @@
     simulation_controllers="$(arg simulation_controllers)"
     robot_description_package="$(arg robot_description_package)"
-    initial_positions_file="(arg initial_positions_file)"
     robot_ip="(arg robot_ip)"
     robot_port="(arg robot_port)"

File: kuka_ros2_control_support/urdf/common_macro.ros2_control.xacro (robot description, xacro)
@@ -9,9 +9,7 @@
                simulation_controllers
                robot_description_package
-               initial_positions_file
                robot_ip
                robot_port"
                >
-      <xacro:property name="initial_positions" value="${load_yaml(initial_positions_file)['initial_positions']}"/>
     <ros2_control name="${name}" type="system">
       <hardware>
@@ -35,5 +33,4 @@
       </hardware>
       <joint name="${prefix}joint_a1">
-        <param name="initial_position">${initial_positions['joint_a1']}</param>
         <command_interface name="position">
           <param name="min">-1</param>
@@ -45,5 +42,4 @@
       </joint>
       <joint name="${prefix}joint_a2">
-        <param name="initial_position">${initial_positions['joint_a2']}</param>
         <command_interface name="position">
           <param name="min">-1</param>
@@ -55,5 +51,4 @@
 	  </joint>
       <joint name="${prefix}joint_a3">
-        <param name="initial_position">${initial_positions['joint_a3']}</param>
         <command_interface name="position">
           <param name="min">-1</param>
@@ -65,5 +60,4 @@
 	  </joint>
       <joint name="${prefix}joint_a4">
-        <param name="initial_position">${initial_positions['joint_a4']}</param>
         <command_interface name="position">
           <param name="min">-1</param>
@@ -75,5 +69,4 @@
       </joint>
       <joint name="${prefix}joint_a5">
-        <param name="initial_position">${initial_positions['joint_a5']}</param>
         <command_interface name="position">
           <param name="min">-1</param>
@@ -85,5 +78,4 @@
       </joint>
       <joint name="${prefix}joint_a6">
-        <param name="initial_position">${initial_positions['joint_a6']}</param>
         <command_interface name="position">
           <param name="min">-1</param>

Commit message: adding initial_positions_file param

File: kuka_ros2_control_support/urdf/common_kuka.xacro (robot description, xacro)
@@ -14,11 +14,12 @@
   <xacro:property name="robot_description_macro_file" value="$(arg robot_description_macro_file)"/>
   <xacro:property name="robot_name" value="$(arg robot_name)"/>
+  <xacro:arg name="initial_positions_file" default="$(find ${robot_description_package})/config/initial_positions.yaml"/>
    <!-- create link fixed to the "world" -->
    <!-- using-external-joints-and-links approach -->
   <link name="world" />
-  <joint name="$(arg prefix)base_joint" type="fixed">
+  <joint name="$(arg prefix)table_link" type="fixed">
     <origin xyz="0 0 0" rpy="0 0 0" />          <!-- position robot in the world -->
     <parent link="world" />
-    <child link="$(arg prefix)base_link"/>
+    <child link="$(arg prefix)table_link"/>
   </joint>
   <xacro:include filename="$(find ${robot_description_package})/urdf/${robot_description_macro_file}"/>
@@ -27,4 +28,5 @@
     name="$(arg robot_name)"
     prefix="$(arg prefix)"
+    initial_positions_file="$(arg initial_positions_file)"
     use_fake_hardware="$(arg use_fake_hardware)"
     sim_gazebo_classic="$(arg sim_gazebo_classic)"
@@ -34,5 +36,5 @@
     robot_ip="(arg robot_ip)"
     robot_port="(arg robot_port)"
-    />
+  />
   <xacro:if value="${robot_description_package == 'kuka_kr3_support'}">
     <xacro:kuka_kr3r540 prefix="$(arg prefix)"/>

File: kuka_ros2_control_support/urdf/common_macro.ros2_control.xacro (robot description, xacro)
@@ -4,4 +4,5 @@
                name
                prefix
+               initial_positions_file
                use_fake_hardware:=^|false
                sim_gazebo_classic:=^|false
@@ -12,4 +13,5 @@
                robot_port"
                >
+    <xacro:property name="initial_positions" value="${load_yaml(initial_positions_file)['initial_positions']}"/>
     <ros2_control name="${name}" type="system">
       <hardware>
@@ -33,4 +35,5 @@
       </hardware>
       <joint name="${prefix}joint_a1">
+        <param name="initial_position">${initial_positions['joint_a1']}</param>
         <command_interface name="position">
           <param name="min">-1</param>
@@ -42,4 +45,5 @@
       </joint>
       <joint name="${prefix}joint_a2">
+        <param name="initial_position">${initial_positions['joint_a2']}</param>
         <command_interface name="position">
           <param name="min">-1</param>
@@ -49,6 +53,7 @@
           <param name="initial_value">0.0</param>
         </state_interface>
-	  </joint>
+	    </joint>
       <joint name="${prefix}joint_a3">
+        <param name="initial_position">${initial_positions['joint_a3']}</param>
         <command_interface name="position">
           <param name="min">-1</param>
@@ -58,6 +63,7 @@
           <param name="initial_value">0.0</param>
         </state_interface>
-	  </joint>
+	    </joint>
       <joint name="${prefix}joint_a4">
+        <param name="initial_position">${initial_positions['joint_a4']}</param>
         <command_interface name="position">
           <param name="min">-1</param>
@@ -69,4 +75,5 @@
       </joint>
       <joint name="${prefix}joint_a5">
+        <param name="initial_position">${initial_positions['joint_a5']}</param>
         <command_interface name="position">
           <param name="min">-1</param>
@@ -78,4 +85,5 @@
       </joint>
       <joint name="${prefix}joint_a6">
+        <param name="initial_position">${initial_positions['joint_a6']}</param>
         <command_interface name="position">
           <param name="min">-1</param>
@@ -88,11 +96,12 @@
       <xacro:if value="${robot_description_package == 'kuka_lbr_iiwa_support'}">
         <joint name="${prefix}joint_a7">
-        <command_interface name="position">
-          <param name="min">-1</param>
-          <param name="max">1</param>
-        </command_interface>
-        <state_interface name="position">
-          <param name="initial_value">0.0</param>
-        </state_interface>
+          <param name="initial_position">${initial_positions['joint_a7']}</param>
+          <command_interface name="position">
+            <param name="min">-1</param>
+            <param name="max">1</param>
+          </command_interface>
+          <state_interface name="position">
+            <param name="initial_value">0.0</param>
+          </state_interface>
         </joint>
       </xacro:if>

Commit message: modified to work with cell description kr10cell and other regular descriptions

File: kuka_ros2_control_support/urdf/common_kuka.xacro (robot description, xacro)
@@ -14,15 +14,38 @@
   <xacro:property name="robot_description_macro_file" value="$(arg robot_description_macro_file)"/>
   <xacro:property name="robot_name" value="$(arg robot_name)"/>
-  <xacro:arg name="initial_positions_file" default="$(find kuka_resources)/config/initial_positions.yaml"/>
-   <!-- create link fixed to the "world" -->
-   <!-- using-external-joints-and-links approach -->
-  <link name="world" />
-  <joint name="$(arg prefix)table_link" type="fixed">
-    <origin xyz="0 0 0" rpy="0 0 0" />          <!-- position robot in the world -->
-    <parent link="world" />
-    <child link="$(arg prefix)table_link"/>
-  </joint>
+  <xacro:if value="${robot_description_package != 'kuka_kr10r1100sixx_cell_description'}">
+    <xacro:arg name="initial_positions_file" default="$(find kuka_resources)/config/initial_positions.yaml"/>
+    <!-- create link fixed to the "world" -->
+    <!-- using-external-joints-and-links approach -->
+    <link name="world" />
+    <joint name="$(arg prefix)base_joint" type="fixed">
+      <origin xyz="0 0 0" rpy="0 0 0" />          <!-- position robot in the world -->
+      <parent link="world" />
+      <child link="$(arg prefix)base_link"/>
+    </joint>
+  </xacro:if>
   <xacro:include filename="$(find ${robot_description_package})/urdf/${robot_description_macro_file}"/>
   <xacro:include filename="$(find kuka_ros2_control_support)/urdf/common_macro.ros2_control.xacro"/>
+  <xacro:if value="${robot_description_package == 'kuka_kr10r1100sixx_cell_description'}">
+    <xacro:arg name="initial_positions_file" default="$(find kuka_kr10r1100sixx_cell_description)/config/initial_positions.yaml"/>
+    <!-- create link fixed to the "world" -->
+    <!-- using-external-joints-and-links approach -->
+    <link name="world" />
+    <joint name="$(arg prefix)table_link" type="fixed">
+      <origin xyz="0 0 0" rpy="0 0 0" />          <!-- position robot in the world -->
+      <parent link="world" />
+      <child link="$(arg prefix)table_link"/>
+    </joint>
+    <xacro:include filename="$(find kuka_kr10r1100sixx_cell_description)/urdf/kr10_macro.ros2_control.xacro"/>
+    <xacro:kr10_gripper_ros2_control name="gripper_control" prefix="$(arg prefix)"/>
+    <xacro:if value="${robot_description_macro_file == 'kr10_cylinder_macro.xacro'}">
+      <xacro:kuka_kr10r1100sixx_cell
+      prefix="$(arg prefix)"
+      robot_ip="(arg robot_ip)"
+      robot_port="(arg robot_port)"
+      use_fake_hardware="$(arg use_fake_hardware)"
+       />
+    </xacro:if>
+  </xacro:if>
   <xacro:kuka_common_ros2_control_macro
     name="$(arg robot_name)"
@@ -37,16 +60,4 @@
     robot_port="(arg robot_port)"
   />
-  <xacro:if value="${robot_description_package == 'kuka_kr10r1100sixx_cell_description'}">
-    <xacro:include filename="$(find kuka_kr10r1100sixx_cell_description)/urdf/kr10_macro.ros2_control.xacro"/>
-    <xacro:kr10_gripper_ros2_control name="gripper_control" prefix="$(arg prefix)"/>
-    <xacro:if value="${robot_description_macro_file == 'kr10_cylinder_macro.xacro'}">
-      <xacro:kuka_kr10r1100sixx_cell
-      prefix="$(arg prefix)"
-      robot_ip="(arg robot_ip)"
-      robot_port="(arg robot_port)"
-      use_fake_hardware="$(arg use_fake_hardware)"
-       />
-    </xacro:if>
-  </xacro:if>
   <xacro:if value="${robot_description_package == 'kuka_kr3_support'}">
     <xacro:kuka_kr3r540 prefix="$(arg prefix)"/>

Commit message: added initial_positions_file arg

File: kuka_ros2_control_support/urdf/common_kuka.xacro (robot description, xacro)
@@ -9,4 +9,5 @@
   <xacro:arg name="robot_description_macro_file" default="kr3r540_macro.xacro"/>
   <xacro:arg name="robot_name" default="kuka_kr3r540"/>
+  <xacro:arg name="initial_positions_file" default="$(find kuka_resources)/config/initial_positions.yaml"/>
   <xacro:property name="robot_description_package" value="$(arg robot_description_package)"/>
   <xacro:property name="robot_description_macro_file" value="$(arg robot_description_macro_file)"/>
@@ -25,4 +26,5 @@
     name="$(arg robot_name)"
     prefix="$(arg prefix)"
+    initial_positions_file="$(arg initial_positions_file)"
     use_mock_hardware="$(arg use_mock_hardware)"
     sim_gazebo_classic="$(arg sim_gazebo_classic)"

File: kuka_ros2_control_support/urdf/common_macro.ros2_control.xacro (robot description, xacro)
@@ -4,4 +4,5 @@
                name
                prefix
+               initial_positions_file
                use_mock_hardware:=^|false
                sim_gazebo_classic:=^|false
@@ -10,4 +11,5 @@
                robot_description_package"
                >
+    <xacro:property name="initial_positions" value="${load_yaml(initial_positions_file)['initial_positions']}"/>
     <ros2_control name="${name}" type="system">
       <hardware>
