Commit message: added kr210r3 cell related for now

File: kuka_ros2_control_support/urdf/common_kuka.xacro (robot description, xacro)
@@ -15,13 +15,15 @@
   <xacro:property name="robot_name" value="$(arg robot_name)"/>
   <xacro:if value="${robot_description_package != 'kuka_kr10r1100sixx_cell_description'}">
-    <xacro:arg name="initial_positions_file" default="$(find kuka_resources)/config/initial_positions.yaml"/>
-    <!-- create link fixed to the "world" -->
-    <!-- using-external-joints-and-links approach -->
-    <link name="world" />
-    <joint name="$(arg prefix)base_joint" type="fixed">
-      <origin xyz="0 0 0" rpy="0 0 0" />          <!-- position robot in the world -->
-      <parent link="world" />
-      <child link="$(arg prefix)base_link"/>
-    </joint>
+    <xacro:if value="${robot_description_package != 'kuka_kr210r3100_cell_description'}">
+      <xacro:arg name="initial_positions_file" default="$(find kuka_resources)/config/initial_positions.yaml"/>
+      <!-- create link fixed to the "world" -->
+      <!-- using-external-joints-and-links approach -->
+      <link name="world" />
+      <joint name="$(arg prefix)base_joint" type="fixed">
+        <origin xyz="0 0 0" rpy="0 0 0" />          <!-- position robot in the world -->
+        <parent link="world" />
+        <child link="$(arg prefix)base_link"/>
+      </joint>
+    </xacro:if>
   </xacro:if>
   <xacro:include filename="$(find ${robot_description_package})/urdf/${robot_description_macro_file}"/>
@@ -46,4 +48,13 @@
       use_fake_hardware="$(arg use_fake_hardware)"
        />
+    </xacro:if>
+  </xacro:if>
+  <xacro:if value="${robot_description_package == 'kuka_kr210r3100_cell_description'}">
+    <xacro:arg name="initial_positions_file" default="$(find kuka_kr210r3100_cell_description)/config/initial_positions.yaml"/>
+    <!-- create link fixed to the "world" -->
+    <!-- using-external-joints-and-links approach -->
+    <link name="world" />
+    <xacro:if value="${robot_description_macro_file == 'kuka_kr210r3100_cell_macro.xacro'}">
+      <xacro:kuka_kr210r3100_cell prefix="$(arg prefix)"/>
     </xacro:if>
   </xacro:if>

Commit message: not needed as removed the kr10 cell pkg

File: kuka_ros2_control_support/urdf/common_kuka.xacro (robot description, xacro)
@@ -27,25 +27,4 @@
   <xacro:include filename="$(find ${robot_description_package})/urdf/${robot_description_macro_file}"/>
   <xacro:include filename="$(find kuka_ros2_control_support)/urdf/common_macro.ros2_control.xacro"/>
-  <xacro:if value="${robot_description_package == 'kuka_kr10r1100sixx_cell_description'}">
-    <xacro:arg name="initial_positions_file" default="$(find kuka_kr10r1100sixx_cell_description)/config/initial_positions.yaml"/>
-    <!-- create link fixed to the "world" -->
-    <!-- using-external-joints-and-links approach -->
-    <link name="world" />
-    <joint name="$(arg prefix)table_link" type="fixed">
-      <origin xyz="0 0 0" rpy="0 0 0" />          <!-- position robot in the world -->
-      <parent link="world" />
-      <child link="$(arg prefix)table_link"/>
-    </joint>
-    <xacro:include filename="$(find kuka_kr10r1100sixx_cell_description)/urdf/kr10_macro.ros2_control.xacro"/>
-    <xacro:kr10_gripper_ros2_control name="gripper_control" prefix="$(arg prefix)"/>
-    <xacro:if value="${robot_description_macro_file == 'kr10_cylinder_macro.xacro'}">
-      <xacro:kuka_kr10r1100sixx_cell
-      prefix="$(arg prefix)"
-      robot_ip="(arg robot_ip)"
-      robot_port="(arg robot_port)"
-      use_fake_hardware="$(arg use_fake_hardware)"
-       />
-    </xacro:if>
-  </xacro:if>
   <xacro:kuka_common_ros2_control_macro
     name="$(arg robot_name)"

Commit message: add control node and rsi

File: kuka_ros2_control_support/urdf/common_kuka.xacro (robot description, xacro)
@@ -1,28 +1,26 @@
 <?xml version="1.0" ?>
-<robot name="$(arg robot_name)" xmlns:xacro="http://wiki.ros.org/xacro">
-  <xacro:arg name="robot_name" default="kuka"/>
+<robot name="kuka" xmlns:xacro="http://wiki.ros.org/xacro">
   <xacro:arg name="prefix" default="" />
-  <xacro:arg name="use_fake_hardware" default="false" />
+  <xacro:arg name="use_mock_hardware" default="false" />
   <xacro:arg name="sim_gazebo_classic" default="false" />
   <xacro:arg name="sim_gazebo" default="false" />
   <xacro:arg name="simulation_controllers" default="" />
-  <xacro:arg name="robot_description_package" default="" />
-  <xacro:arg name="robot_description_macro_file" default="" />
-  <xacro:arg name="robot_ip" default="172.0.0.1"/>
-  <xacro:arg name="robot_port" default="49152"/>
+  <xacro:arg name="robot_description_package" default="kuka_kr3_support"/>
+  <xacro:arg name="robot_description_macro_file" default="kr3r540_macro.xacro"/>
+  <xacro:arg name="robot_name" default="kuka_kr3r540"/>
+  <xacro:arg name="initial_positions_file" default="$(find kuka_resources)/config/initial_positions.yaml"/>
+  <xacro:arg name="listen_ip_address" default="127.0.0.1" />
+  <xacro:arg name="listen_port" default="49152" />
   <xacro:property name="robot_description_package" value="$(arg robot_description_package)"/>
   <xacro:property name="robot_description_macro_file" value="$(arg robot_description_macro_file)"/>
   <xacro:property name="robot_name" value="$(arg robot_name)"/>
-  <xacro:if value="${robot_description_package != 'kuka_kr10r1100sixx_cell_description'}">
-    <xacro:arg name="initial_positions_file" default="$(find kuka_resources)/config/initial_positions.yaml"/>
-    <!-- create link fixed to the "world" -->
-    <!-- using-external-joints-and-links approach -->
-    <link name="world" />
-    <joint name="$(arg prefix)base_joint" type="fixed">
-      <origin xyz="0 0 0" rpy="0 0 0" />          <!-- position robot in the world -->
-      <parent link="world" />
-      <child link="$(arg prefix)base_link"/>
-    </joint>
-  </xacro:if>
+   <!-- create link fixed to the "world" -->
+   <!-- using-external-joints-and-links approach -->
+  <link name="world" />
+  <joint name="$(arg prefix)base_joint" type="fixed">
+    <origin xyz="0 0 0" rpy="0 0 0" />          <!-- position robot in the world -->
+    <parent link="world" />
+    <child link="$(arg prefix)base_link"/>
+  </joint>
   <xacro:include filename="$(find ${robot_description_package})/urdf/${robot_description_macro_file}"/>
   <xacro:include filename="$(find kuka_ros2_control_support)/urdf/common_macro.ros2_control.xacro"/>
@@ -31,12 +29,12 @@
     prefix="$(arg prefix)"
     initial_positions_file="$(arg initial_positions_file)"
-    use_fake_hardware="$(arg use_fake_hardware)"
+    use_mock_hardware="$(arg use_mock_hardware)"
     sim_gazebo_classic="$(arg sim_gazebo_classic)"
     sim_gazebo="$(arg sim_gazebo)"
     simulation_controllers="$(arg simulation_controllers)"
     robot_description_package="$(arg robot_description_package)"
-    robot_ip="(arg robot_ip)"
-    robot_port="(arg robot_port)"
-  />
+    listen_ip_address="$(arg listen_ip_address)"
+    listen_port="$(arg listen_port)"
+    />
   <xacro:if value="${robot_description_package == 'kuka_kr3_support'}">
     <xacro:kuka_kr3r540 prefix="$(arg prefix)"/>
@@ -82,10 +80,5 @@
   </xacro:if>
   <xacro:if value="${robot_description_package == 'kuka_kr210_support'}">
-    <xacro:if value="${robot_description_macro_file == 'kr210l150_macro.xacro'}">
-      <xacro:kuka_kr210l150 prefix="$(arg prefix)"/>
-    </xacro:if>
-    <xacro:if value="${robot_description_macro_file == 'kr210r3100_macro.xacro'}">
-      <xacro:kuka_kr210r3100 prefix="$(arg prefix)"/>
-    </xacro:if>
+    <xacro:kuka_kr210l150 prefix="$(arg prefix)"/>
   </xacro:if>
   <xacro:if value="${robot_description_package == 'kuka_lbr_iiwa_support'}">

File: kuka_ros2_control_support/urdf/common_macro.ros2_control.xacro (robot description, xacro)
@@ -5,23 +5,18 @@
                prefix
                initial_positions_file
-               use_fake_hardware:=^|false
+               use_mock_hardware:=^|false
                sim_gazebo_classic:=^|false
                sim_gazebo:=^|false
                simulation_controllers
                robot_description_package
-               robot_ip
-               robot_port"
+               listen_ip_address:=^|127.0.0.1
+               listen_port:=^|49152"
                >
-    <xacro:property name="initial_positions" value="${xacro.load_yaml(initial_positions_file)['initial_positions']}"/>
+    <xacro:property name="initial_positions" value="${load_yaml(initial_positions_file)['initial_positions']}"/>
     <ros2_control name="${name}" type="system">
       <hardware>
-        <xacro:if value="${use_fake_hardware}">
-          <plugin>fake_components/GenericSystem</plugin>
+        <xacro:if value="${use_mock_hardware}">
+          <plugin>mock_components/GenericSystem</plugin>
         </xacro:if>
-        <xacro:unless value="${use_fake_hardware}">
-            <plugin>kuka_eki_hw_interface/KukaEkiHardwareInterface</plugin>
-            <param name="robot_ip">${robot_ip}</param>
-            <param name="robot_port">${robot_port}</param>
-        </xacro:unless>
         <xacro:if value="${sim_gazebo_classic}">
           <plugin>gazebo_ros2_control/GazeboSystem</plugin>
@@ -30,10 +25,11 @@
           <plugin>ign_ros2_control/IgnitionSystem</plugin>
         </xacro:if>
-        <xacro:unless value="${use_fake_hardware or sim_gazebo_classic or sim_gazebo}">
-          <plugin>robot_hardware_inteface/RobotHardwareInteface</plugin>
+        <xacro:unless value="${use_mock_hardware or sim_gazebo_classic or sim_gazebo}">
+          <plugin>kuka_rsi_hw_interface/KukaSystemPositionOnlyHardware</plugin>
+          <param name="listen_address">${listen_ip_address}</param>
+          <param name="listen_port">${listen_port}</param>
         </xacro:unless>
       </hardware>
       <joint name="${prefix}joint_a1">
-        <param name="initial_position">${initial_positions['joint_a1']}</param>
         <command_interface name="position">
           <param name="min">-1</param>
@@ -45,5 +41,4 @@
       </joint>
       <joint name="${prefix}joint_a2">
-        <param name="initial_position">${initial_positions['joint_a2']}</param>
         <command_interface name="position">
           <param name="min">-1</param>
@@ -53,7 +48,6 @@
           <param name="initial_value">0.0</param>
         </state_interface>
-	    </joint>
+	  </joint>
       <joint name="${prefix}joint_a3">
-        <param name="initial_position">${initial_positions['joint_a3']}</param>
         <command_interface name="position">
           <param name="min">-1</param>
@@ -63,7 +57,6 @@
           <param name="initial_value">0.0</param>
         </state_interface>
-	    </joint>
+	  </joint>
       <joint name="${prefix}joint_a4">
-        <param name="initial_position">${initial_positions['joint_a4']}</param>
         <command_interface name="position">
           <param name="min">-1</param>
@@ -75,5 +68,4 @@
       </joint>
       <joint name="${prefix}joint_a5">
-        <param name="initial_position">${initial_positions['joint_a5']}</param>
         <command_interface name="position">
           <param name="min">-1</param>
@@ -85,5 +77,4 @@
       </joint>
       <joint name="${prefix}joint_a6">
-        <param name="initial_position">${initial_positions['joint_a6']}</param>
         <command_interface name="position">
           <param name="min">-1</param>
@@ -96,12 +87,11 @@
       <xacro:if value="${robot_description_package == 'kuka_lbr_iiwa_support'}">
         <joint name="${prefix}joint_a7">
-          <param name="initial_position">${initial_positions['joint_a7']}</param>
-          <command_interface name="position">
-            <param name="min">-1</param>
-            <param name="max">1</param>
-          </command_interface>
-          <state_interface name="position">
-            <param name="initial_value">0.0</param>
-          </state_interface>
+        <command_interface name="position">
+          <param name="min">-1</param>
+          <param name="max">1</param>
+        </command_interface>
+        <state_interface name="position">
+          <param name="initial_value">0.0</param>
+        </state_interface>
         </joint>
       </xacro:if>

Commit message: arg for origin of robo

File: kuka_ros2_control_support/urdf/common_kuka.xacro (robot description, xacro)
@@ -2,4 +2,5 @@
 <robot name="kuka" xmlns:xacro="http://wiki.ros.org/xacro">
   <xacro:arg name="prefix" default="" />
+  <xacro:arg name="origin" default="0 0 0" />
   <xacro:arg name="use_mock_hardware" default="false" />
   <xacro:arg name="sim_gazebo_classic" default="false" />
@@ -19,5 +20,5 @@
   <link name="world" />
   <joint name="$(arg prefix)base_joint" type="fixed">
-    <origin xyz="0 0 0" rpy="0 0 0" />          <!-- position robot in the world -->
+    <origin xyz="$(arg origin)" rpy="0 0 0" />          <!-- position robot in the world -->
     <parent link="world" />
     <child link="$(arg prefix)base_link"/>
