Commit message: common xacro and ros2_controlxacro

File: kuka_ros2_control_support/urdf/common_macro.ros2_control.xacro (robot description, xacro)
@@ -1,10 +1,28 @@
 <?xml version="1.0"?>
 <robot xmlns:xacro="http://www.ros.org/wiki/xacro">
-  <xacro:macro name="kuka_common_ros2_control_macro" params="name prefix use_mock_hardware:=^|false">
+  <xacro:macro name="kuka_common_ros2_control_macro" params="
+               name
+               prefix
+               use_mock_hardware:=^|false
+               mock_sensor_commands:=^|false
+               sim_gazebo_classic:=^|false
+               sim_gazebo:=^|false
+               simulation_controllers"
+               >
     <ros2_control name="${name}" type="system">
       <hardware>
         <xacro:if value="${use_mock_hardware}">
           <plugin>mock_components/GenericSystem</plugin>
+          <param name="mock_sensor_commands">${mock_sensor_commands}</param>
         </xacro:if>
+        <xacro:if value="${sim_gazebo_classic}">
+          <plugin>gazebo_ros2_control/GazeboSystem</plugin>
+        </xacro:if>
+        <xacro:if value="${sim_gazebo}">
+          <plugin>ign_ros2_control/IgnitionSystem</plugin>
+        </xacro:if>
+        <xacro:unless value="${use_mock_hardware or sim_gazebo_classic or sim_gazebo}">
+          <plugin>robot_hardware_inteface/RobotHardwareInteface</plugin>
+        </xacro:unless>
       </hardware>
       <joint name="${prefix}joint_a1">
@@ -62,5 +80,47 @@
         </state_interface>
       </joint>
+      <sensor name="tcp_fts_sensor">            <!-- Remove/change sensors as needed -->
+        <state_interface name="fx"/>
+        <state_interface name="fy"/>
+        <state_interface name="fz"/>
+        <state_interface name="tx"/>
+        <state_interface name="ty"/>
+        <state_interface name="tz"/>
+        <param name="frame_id">tool0</param>    <!-- Change sensors as needed -->
+        <param name="min_fx">-100</param>
+        <param name="max_fx">100</param>
+        <param name="min_fy">-100</param>
+        <param name="max_fy">100</param>
+        <param name="min_fz">-200</param>
+        <param name="max_fz">200</param>
+        <param name="min_tx">-10</param>
+        <param name="max_tx">10</param>
+        <param name="min_ty">-10</param>
+        <param name="max_ty">10</param>
+        <param name="min_tz">-15</param>
+        <param name="max_tz">15</param>
+      </sensor>
     </ros2_control>
+    <xacro:if value="$(arg sim_gazebo_classic)">
+      <!-- Gazebo plugins -->
+      <gazebo reference="world">
+      </gazebo>
+      <gazebo>
+        <plugin filename="libgazebo_ros2_control.so" name="gazebo_ros2_control">
+          <parameters>${simulation_controllers}</parameters>
+        </plugin>
+      </gazebo>
+    </xacro:if>
+    <xacro:if value="$(arg sim_gazebo)">
+      <!-- Gazebo plugins -->
+      <gazebo reference="world">
+      </gazebo>
+      <gazebo>
+        <plugin filename="libign_ros2_control-system.so" name="ign_ros2_control::IgnitionROS2ControlPlugin">
+          <parameters>${simulation_controllers}</parameters>
+          <controller_manager_node_name>${prefix}controller_manager</controller_manager_node_name>
+        </plugin>
+      </gazebo>
+    </xacro:if>
   </xacro:macro>
 </robot>

Commit message: functional ros2_control support for kuka base models

File: kuka_ros2_control_support/urdf/common_macro.ros2_control.xacro (robot description, xacro)
@@ -1,5 +1,8 @@
 <?xml version="1.0"?>
 <robot xmlns:xacro="http://www.ros.org/wiki/xacro">
-  <xacro:macro name="kuka_common_ros2_control_macro" params="name prefix use_mock_hardware:=^|false">
+  <xacro:macro name="kuka_common_ros2_control_macro" params="
+               name
+               prefix
+               use_mock_hardware:=^|false">
     <ros2_control name="${name}" type="system">
       <hardware>

Commit message: correction

File: kuka_ros2_control_support/urdf/common_macro.ros2_control.xacro (robot description, xacro)
@@ -28,5 +28,5 @@
           <param name="initial_value">0.0</param>
         </state_interface>
-	  </joint>
+	    </joint>
       <joint name="${prefix}joint_a3">
         <command_interface name="position">
@@ -37,5 +37,5 @@
           <param name="initial_value">0.0</param>
         </state_interface>
-	  </joint>
+	    </joint>
       <joint name="${prefix}joint_a4">
         <command_interface name="position">

Commit message: Update kuka_ros2_control_support/urdf/common_macro.ros2_control.xacro

File: kuka_ros2_control_support/urdf/common_macro.ros2_control.xacro (robot description, xacro)
@@ -28,5 +28,5 @@
           <param name="initial_value">0.0</param>
         </state_interface>
-	    </joint>
+	   </joint>
       <joint name="${prefix}joint_a3">
         <command_interface name="position">

Commit message: Apply suggestions from code review

File: kuka_ros2_control_support/urdf/common_macro.ros2_control.xacro (robot description, xacro)
@@ -28,5 +28,5 @@
           <param name="initial_value">0.0</param>
         </state_interface>
-	   </joint>
+	  </joint>
       <joint name="${prefix}joint_a3">
         <command_interface name="position">
@@ -37,5 +37,5 @@
           <param name="initial_value">0.0</param>
         </state_interface>
-	    </joint>
+	  </joint>
       <joint name="${prefix}joint_a4">
         <command_interface name="position">

Commit message: added kuka_ros2_control_support along side kuka_ros2_control_sim_support

File: kuka_ros2_control_support/urdf/common_macro.ros2_control.xacro (robot description, xacro)
@@ -1,10 +1,27 @@
 <?xml version="1.0"?>
 <robot xmlns:xacro="http://www.ros.org/wiki/xacro">
-  <xacro:macro name="kuka_common_ros2_control_macro" params="name prefix use_mock_hardware:=^|false">
+  <xacro:macro name="kuka_common_ros2_control_macro" params="
+               name
+               prefix
+               use_mock_hardware:=^|false
+               sim_gazebo_classic:=^|false
+               sim_gazebo:=^|false
+               simulation_controllers
+               robot_description_package"
+               >
     <ros2_control name="${name}" type="system">
       <hardware>
         <xacro:if value="${use_mock_hardware}">
-          <plugin>fake_components/GenericSystem</plugin>
+          <plugin>mock_components/GenericSystem</plugin>
         </xacro:if>
+        <xacro:if value="${sim_gazebo_classic}">
+          <plugin>gazebo_ros2_control/GazeboSystem</plugin>
+        </xacro:if>
+        <xacro:if value="${sim_gazebo}">
+          <plugin>ign_ros2_control/IgnitionSystem</plugin>
+        </xacro:if>
+        <xacro:unless value="${use_mock_hardware or sim_gazebo_classic or sim_gazebo}">
+          <plugin>robot_hardware_inteface/RobotHardwareInteface</plugin>
+        </xacro:unless>
       </hardware>
       <joint name="${prefix}joint_a1">
@@ -62,5 +79,37 @@
         </state_interface>
       </joint>
+      <xacro:if value="${robot_description_package == 'kuka_lbr_iiwa_support'}">
+        <joint name="${prefix}joint_a7">
+        <command_interface name="position">
+          <param name="min">-1</param>
+          <param name="max">1</param>
+        </command_interface>
+        <state_interface name="position">
+          <param name="initial_value">0.0</param>
+        </state_interface>
+        </joint>
+      </xacro:if>
     </ros2_control>
+    <xacro:if value="$(arg sim_gazebo_classic)">
+      <!-- Gazebo plugins -->
+      <gazebo reference="world">
+      </gazebo>
+      <gazebo>
+        <plugin filename="libgazebo_ros2_control.so" name="gazebo_ros2_control">
+          <parameters>${simulation_controllers}</parameters>
+        </plugin>
+      </gazebo>
+    </xacro:if>
+    <xacro:if value="$(arg sim_gazebo)">
+      <!-- Gazebo plugins -->
+      <gazebo reference="world">
+      </gazebo>
+      <gazebo>
+        <plugin filename="libign_ros2_control-system.so" name="ign_ros2_control::IgnitionROS2ControlPlugin">
+          <parameters>${simulation_controllers}</parameters>
+          <controller_manager_node_name>${prefix}controller_manager</controller_manager_node_name>
+        </plugin>
+      </gazebo>
+    </xacro:if>
   </xacro:macro>
 </robot>

Commit message: updated with initial_positions, robot_ip, robot_port args

File: kuka_ros2_control_support/urdf/common_macro.ros2_control.xacro (robot description, xacro)
@@ -8,6 +8,10 @@
                sim_gazebo:=^|false
                simulation_controllers
-               robot_description_package"
+               robot_description_package
+               initial_positions_file
+               robot_ip
+               robot_port"
                >
+      <xacro:property name="initial_positions" value="${load_yaml(initial_positions_file)['initial_positions']}"/>
     <ros2_control name="${name}" type="system">
       <hardware>
@@ -15,4 +19,9 @@
           <plugin>fake_components/GenericSystem</plugin>
         </xacro:if>
+        <xacro:unless value="${use_fake_hardware}">
+            <plugin>kuka_eki_hw_interface/KukaEkiHardwareInterface</plugin>
+            <param name="robot_ip">${robot_ip}</param>
+            <param name="robot_port">${robot_port}</param>
+        </xacro:unless>
         <xacro:if value="${sim_gazebo_classic}">
           <plugin>gazebo_ros2_control/GazeboSystem</plugin>
@@ -26,4 +35,5 @@
       </hardware>
       <joint name="${prefix}joint_a1">
+        <param name="initial_position">${initial_positions['joint_a1']}</param>
         <command_interface name="position">
           <param name="min">-1</param>
@@ -35,4 +45,5 @@
       </joint>
       <joint name="${prefix}joint_a2">
+        <param name="initial_position">${initial_positions['joint_a2']}</param>
         <command_interface name="position">
           <param name="min">-1</param>
@@ -44,4 +55,5 @@
 	  </joint>
       <joint name="${prefix}joint_a3">
+        <param name="initial_position">${initial_positions['joint_a3']}</param>
         <command_interface name="position">
           <param name="min">-1</param>
@@ -53,4 +65,5 @@
 	  </joint>
       <joint name="${prefix}joint_a4">
+        <param name="initial_position">${initial_positions['joint_a4']}</param>
         <command_interface name="position">
           <param name="min">-1</param>
@@ -62,4 +75,5 @@
       </joint>
       <joint name="${prefix}joint_a5">
+        <param name="initial_position">${initial_positions['joint_a5']}</param>
         <command_interface name="position">
           <param name="min">-1</param>
@@ -71,4 +85,5 @@
       </joint>
       <joint name="${prefix}joint_a6">
+        <param name="initial_position">${initial_positions['joint_a6']}</param>
         <command_interface name="position">
           <param name="min">-1</param>

Commit message: ros2_control support pkg files

File: kuka_ros2_control_support/urdf/common_macro.ros2_control.xacro (robot description, xacro)
@@ -13,5 +13,5 @@
                robot_port"
                >
-    <xacro:property name="initial_positions" value="${load_yaml(initial_positions_file)['initial_positions']}"/>
+    <xacro:property name="initial_positions" value="${xacro.load_yaml(initial_positions_file)['initial_positions']}"/>
     <ros2_control name="${name}" type="system">
       <hardware>

Commit message: Some cleanups.

File: kuka_ros2_control_support/urdf/common_macro.ros2_control.xacro (robot description, xacro)
@@ -4,14 +4,17 @@
                name
                prefix
-               initial_positions_file
+               use_eki_communication:=^|false
+               eki_robot_ip:=^|127.0.0.1
+               eki_robot_port:=^|54600
+               use_rsi_communication:=^|false
+               rsi_listen_ip:=^|127.0.0.1
+               rsi_listen_port:=^|49152
                use_mock_hardware:=^|false
                sim_gazebo_classic:=^|false
                sim_gazebo:=^|false
                simulation_controllers
-               robot_description_package
-               listen_ip_address:=^|127.0.0.1
-               listen_port:=^|49152"
+               description_package
+               initial_positions:=${dict(joint_a1=0.0,joint_a2=-1.57,joint_a3=1.57,joint_a4=0.0,joint_a5=1.57,joint_a6=0.0)}"
                >
-    <xacro:property name="initial_positions" value="${load_yaml(initial_positions_file)['initial_positions']}"/>
     <ros2_control name="${name}" type="system">
       <hardware>
@@ -25,9 +28,14 @@
           <plugin>ign_ros2_control/IgnitionSystem</plugin>
         </xacro:if>
-        <xacro:unless value="${use_mock_hardware or sim_gazebo_classic or sim_gazebo}">
-          <plugin>kuka_rsi_hw_interface/KukaSystemPositionOnlyHardware</plugin>
-          <param name="listen_address">${listen_ip_address}</param>
-          <param name="listen_port">${listen_port}</param>
-        </xacro:unless>
+        <xacro:if value="${use_eki_communication}">
+          <plugin>kuka_eki_hw_interface/RobotControlInterface</plugin>
+          <param name="robot_ip">${eki_robot_ip}</param>
+          <param name="robot_port">${eki_robot_port}</param>
+        </xacro:if>
+        <xacro:if value="${use_rsi_communication}">
+          <plugin>kuka_rsi_hw_interface/RobotControlnterface</plugin>
+          <param name="listen_address">${rsi_listen_ip}</param>
+          <param name="listen_port">${rsi_listen_port}</param>
+        </xacro:if>
       </hardware>
       <joint name="${prefix}joint_a1">
@@ -37,5 +45,5 @@
         </command_interface>
         <state_interface name="position">
-          <param name="initial_value">0.0</param>
+          <param name="initial_value">${initial_positions['joint_a1']}</param>
         </state_interface>
       </joint>
@@ -46,5 +54,5 @@
         </command_interface>
         <state_interface name="position">
-          <param name="initial_value">0.0</param>
+          <param name="initial_value">${initial_positions['joint_a2']}</param>
         </state_interface>
 	  </joint>
@@ -55,5 +63,5 @@
         </command_interface>
         <state_interface name="position">
-          <param name="initial_value">0.0</param>
+          <param name="initial_value">${initial_positions['joint_a3']}</param>
         </state_interface>
 	  </joint>
@@ -64,5 +72,5 @@
         </command_interface>
         <state_interface name="position">
-          <param name="initial_value">0.0</param>
+          <param name="initial_value">${initial_positions['joint_a4']}</param>
         </state_interface>
       </joint>
@@ -73,5 +81,5 @@
         </command_interface>
         <state_interface name="position">
-          <param name="initial_value">0.0</param>
+          <param name="initial_value">${initial_positions['joint_a5']}</param>
         </state_interface>
       </joint>
@@ -82,8 +90,8 @@
         </command_interface>
         <state_interface name="position">
-          <param name="initial_value">0.0</param>
+          <param name="initial_value">${initial_positions['joint_a6']}</param>
         </state_interface>
       </joint>
-      <xacro:if value="${robot_description_package == 'kuka_lbr_iiwa_support'}">
+      <xacro:if value="${description_package == 'kuka_lbr_iiwa_support'}">
         <joint name="${prefix}joint_a7">
         <command_interface name="position">
@@ -92,5 +100,5 @@
         </command_interface>
         <state_interface name="position">
-          <param name="initial_value">0.0</param>
+          <param name="initial_value">${initial_positions['joint_a7']}</param>
         </state_interface>
         </joint>
