Commit message: Renamed package, adjust compilation for different robots and setups. Use common `.srdf` file for all robots. Restructure how ros2_control URDF is used.

File: kuka_ros2_control_support/urdf/common_kuka.xacro (robot description, xacro)
@@ -1,86 +1,94 @@
 <?xml version="1.0" ?>
-<robot name="kuka" xmlns:xacro="http://wiki.ros.org/xacro">
+<robot name="$(arg robot_name)" xmlns:xacro="http://wiki.ros.org/xacro">
+  <xacro:arg name="robot_name" default="kuka" />
   <xacro:arg name="prefix" default="" />
+  <xacro:arg name="description_package" default="" />
+  <xacro:arg name="description_macro_file" default="" />
+  <xacro:arg name="use_eki_communication" default="false" />
+  <xacro:arg name="eki_robot_ip" default="127.0.0.1" />
+  <xacro:arg name="eki_robot_port" default="54600" />
+  <xacro:arg name="use_rsi_communication" default="false" />
+  <xacro:arg name="rsi_listen_ip" default="127.0.0.1" />
+  <xacro:arg name="rsi_listen_port" default="49152" />
+  <!-- ros2_control mock and simulation plugins -->
   <xacro:arg name="use_mock_hardware" default="false" />
   <xacro:arg name="sim_gazebo_classic" default="false" />
   <xacro:arg name="sim_gazebo" default="false" />
   <xacro:arg name="simulation_controllers" default="" />
-  <xacro:arg name="robot_description_package" default="kuka_kr3_support"/>
-  <xacro:arg name="robot_description_macro_file" default="kr3r540_macro.xacro"/>
-  <xacro:arg name="robot_name" default="kuka_kr3r540"/>
   <xacro:arg name="initial_positions_file" default="$(find kuka_resources)/config/initial_positions.yaml"/>
-  <xacro:arg name="listen_ip_address" default="127.0.0.1" />
-  <xacro:arg name="listen_port" default="49152" />
-  <xacro:property name="robot_description_package" value="$(arg robot_description_package)"/>
-  <xacro:property name="robot_description_macro_file" value="$(arg robot_description_macro_file)"/>
+  <xacro:property name="description_package" value="$(arg description_package)"/>
+  <xacro:property name="description_macro_file" value="$(arg description_macro_file)"/>
   <xacro:property name="robot_name" value="$(arg robot_name)"/>
-   <!-- create link fixed to the "world" -->
-   <!-- using-external-joints-and-links approach -->
-  <link name="world" />
-  <joint name="$(arg prefix)base_joint" type="fixed">
-    <origin xyz="0 0 0" rpy="0 0 0" />          <!-- position robot in the world -->
-    <parent link="world" />
-    <child link="$(arg prefix)base_link"/>
-  </joint>
-  <xacro:include filename="$(find ${robot_description_package})/urdf/${robot_description_macro_file}"/>
+  <!-- convert to property to use substitution in function -->
+  <xacro:property name="initial_positions_file" default="$(arg initial_positions_file)"/>
+  <xacro:include filename="$(find ${description_package})/urdf/${description_macro_file}"/>
   <xacro:include filename="$(find kuka_ros2_control_support)/urdf/common_macro.ros2_control.xacro"/>
   <xacro:kuka_common_ros2_control_macro
     name="$(arg robot_name)"
     prefix="$(arg prefix)"
-    initial_positions_file="$(arg initial_positions_file)"
+    use_eki_communication="$(arg use_eki_communication)"
+    eki_robot_ip="$(arg eki_robot_ip)"
+    eki_robot_port="$(arg eki_robot_port)"
+    use_rsi_communication="$(arg use_rsi_communication)"
+    rsi_listen_ip="$(arg rsi_listen_ip)"
+    rsi_listen_port="$(arg rsi_listen_port)"
     use_mock_hardware="$(arg use_mock_hardware)"
     sim_gazebo_classic="$(arg sim_gazebo_classic)"
     sim_gazebo="$(arg sim_gazebo)"
     simulation_controllers="$(arg simulation_controllers)"
-    robot_description_package="$(arg robot_description_package)"
-    listen_ip_address="$(arg listen_ip_address)"
-    listen_port="$(arg listen_port)"
-    />
-  <xacro:if value="${robot_description_package == 'kuka_kr3_support'}">
+    description_package="$(arg description_package)"
+    initial_positions="${xacro.load_yaml(initial_positions_file)}"
+  />
+  <xacro:if value="${description_package == 'kuka_kr3_support'}">
     <xacro:kuka_kr3r540 prefix="$(arg prefix)"/>
   </xacro:if>
-  <xacro:if value="${robot_description_package == 'kuka_kr5_support'}">
+  <xacro:if value="${description_package == 'kuka_kr5_support'}">
     <xacro:kuka_kr5_arc prefix="$(arg prefix)"/>
   </xacro:if>
-  <xacro:if value="${robot_description_package == 'kuka_kr6_support'}">
-    <xacro:if value="${robot_description_macro_file == 'kr6r700sixx_macro.xacro'}">
+  <xacro:if value="${description_package == 'kuka_kr6_support'}">
+    <xacro:if value="${description_macro_file == 'kr6r700sixx_macro.xacro'}">
       <xacro:kuka_kr6r700sixx prefix="$(arg prefix)"/>
     </xacro:if>
-    <xacro:if value="${robot_description_macro_file == 'kr6r900_2_macro.xacro'}">
+    <xacro:if value="${description_macro_file == 'kr6r900_2_macro.xacro'}">
       <xacro:kuka_kr6r900_2 prefix="$(arg prefix)"/>
     </xacro:if>
-    <xacro:if value="${robot_description_macro_file == 'kr6r900sixx_macro.xacro'}">
+    <xacro:if value="${description_macro_file == 'kr6r900sixx_macro.xacro'}">
       <xacro:kuka_kr6r900sixx prefix="$(arg prefix)"/>
     </xacro:if>
   </xacro:if>
-  <xacro:if value="${robot_description_package == 'kuka_kr10_support'}">
-    <xacro:if value="${robot_description_macro_file == 'kr10r900_2_macro.xacro'}">
+  <xacro:if value="${description_package == 'kuka_kr10_support'}">
+    <xacro:if value="${description_macro_file == 'kr10r900_2_macro.xacro'}">
       <xacro:kuka_kr10r900_2 prefix="$(arg prefix)"/>
     </xacro:if>
-    <xacro:if value="${robot_description_macro_file == 'kr10r1100sixx_macro.xacro'}">
+    <xacro:if value="${description_macro_file == 'kr10r1100sixx_macro.xacro'}">
       <xacro:kuka_kr10r1100sixx prefix="$(arg prefix)"/>
     </xacro:if>
-    <xacro:if value="${robot_description_macro_file == 'kr10r1420_macro.xacro'}">
+    <xacro:if value="${description_macro_file == 'kr10r1420_macro.xacro'}">
       <xacro:kuka_kr10r1420 prefix="$(arg prefix)"/>
     </xacro:if>
   </xacro:if>
-  <xacro:if value="${robot_description_package == 'kuka_kr16_support'}">
+  <xacro:if value="${description_package == 'kuka_kr16_support'}">
     <xacro:kuka_kr16_2 prefix="$(arg prefix)"/>
   </xacro:if>
-  <xacro:if value="${robot_description_package == 'kuka_kr120_support'}">
+  <xacro:if value="${description_package == 'kuka_kr120_support'}">
     <xacro:kuka_kr120r2500pro prefix="$(arg prefix)"/>
   </xacro:if>
-  <xacro:if value="${robot_description_package == 'kuka_kr150_support'}">
-    <xacro:if value="${robot_description_macro_file == 'kr150_2_macro.xacro'}">
+  <xacro:if value="${description_package == 'kuka_kr150_support'}">
+    <xacro:if value="${description_macro_file == 'kr150_2_macro.xacro'}">
       <xacro:kuka_kr150_2 prefix="$(arg prefix)"/>
     </xacro:if>
-    <xacro:if value="${robot_description_macro_file == 'kr150r3100_2_macro.xacro'}">
+    <xacro:if value="${description_macro_file == 'kr150r3100_2_macro.xacro'}">
       <xacro:kuka_kr150r3100_2 prefix="$(arg prefix)"/>
     </xacro:if>
   </xacro:if>
-  <xacro:if value="${robot_description_package == 'kuka_kr210_support'}">
-    <xacro:kuka_kr210l150 prefix="$(arg prefix)"/>
+  <xacro:if value="${description_package == 'kuka_kr210_support'}">
+    <xacro:if value="${description_macro_file == 'kr210l150_macro.xacro'}">
+      <xacro:kuka_kr210l150 prefix="$(arg prefix)"/>
+    </xacro:if>
+    <xacro:if value="${description_macro_file == 'kr210r3100_macro.xacro'}">
+      <xacro:kuka_kr210r3100 prefix="$(arg prefix)"/>
+    </xacro:if>
   </xacro:if>
-  <xacro:if value="${robot_description_package == 'kuka_lbr_iiwa_support'}">
+  <xacro:if value="${description_package == 'kuka_lbr_iiwa_support'}">
     <xacro:kuka_lbr_iiwa_14_r820 prefix="$(arg prefix)"/>
   </xacro:if>

File: kuka_ros2_control_support/urdf/common_macro.ros2_control.xacro (robot description, xacro)
@@ -4,14 +4,17 @@
                name
                prefix
-               initial_positions_file
+               use_eki_communication:=^|false
+               eki_robot_ip:=^|127.0.0.1
+               eki_robot_port:=^|54600
+               use_rsi_communication:=^|false
+               rsi_listen_ip:=^|127.0.0.1
+               rsi_listen_port:=^|49152
                use_mock_hardware:=^|false
                sim_gazebo_classic:=^|false
                sim_gazebo:=^|false
                simulation_controllers
-               robot_description_package
-               listen_ip_address:=^|127.0.0.1
-               listen_port:=^|49152"
+               description_package
+               initial_positions:=${dict(joint_a1=0.0,joint_a2=-1.57,joint_a3=1.57,joint_a4=0.0,joint_a5=1.57,joint_a6=0.0)}"
                >
-    <xacro:property name="initial_positions" value="${load_yaml(initial_positions_file)['initial_positions']}"/>
     <ros2_control name="${name}" type="system">
       <hardware>
@@ -25,9 +28,14 @@
           <plugin>ign_ros2_control/IgnitionSystem</plugin>
         </xacro:if>
-        <xacro:unless value="${use_mock_hardware or sim_gazebo_classic or sim_gazebo}">
-          <plugin>kuka_rsi_hw_interface/KukaSystemPositionOnlyHardware</plugin>
-          <param name="listen_address">${listen_ip_address}</param>
-          <param name="listen_port">${listen_port}</param>
-        </xacro:unless>
+        <xacro:if value="${use_eki_communication}">
+          <plugin>kuka_eki_hw_interface/RobotControl</plugin>
+          <param name="robot_ip">${eki_robot_ip}</param>
+          <param name="robot_port">${eki_robot_port}</param>
+        </xacro:if>
+        <xacro:if value="${use_rsi_communication}">
+          <plugin>kuka_rsi_hw_interface/OnlyRobotControl</plugin>
+          <param name="listen_address">${rsi_listen_ip}</param>
+          <param name="listen_port">${rsi_listen_port}</param>
+        </xacro:if>
       </hardware>
       <joint name="${prefix}joint_a1">
@@ -37,5 +45,5 @@
         </command_interface>
         <state_interface name="position">
-          <param name="initial_value">0.0</param>
+          <param name="initial_value">${initial_positions['joint_a1']}</param>
         </state_interface>
       </joint>
@@ -46,5 +54,5 @@
         </command_interface>
         <state_interface name="position">
-          <param name="initial_value">0.0</param>
+          <param name="initial_value">${initial_positions['joint_a2']}</param>
         </state_interface>
 	  </joint>
@@ -55,5 +63,5 @@
         </command_interface>
         <state_interface name="position">
-          <param name="initial_value">0.0</param>
+          <param name="initial_value">${initial_positions['joint_a3']}</param>
         </state_interface>
 	  </joint>
@@ -64,5 +72,5 @@
         </command_interface>
         <state_interface name="position">
-          <param name="initial_value">0.0</param>
+          <param name="initial_value">${initial_positions['joint_a4']}</param>
         </state_interface>
       </joint>
@@ -73,5 +81,5 @@
         </command_interface>
         <state_interface name="position">
-          <param name="initial_value">0.0</param>
+          <param name="initial_value">${initial_positions['joint_a5']}</param>
         </state_interface>
       </joint>
@@ -82,8 +90,8 @@
         </command_interface>
         <state_interface name="position">
-          <param name="initial_value">0.0</param>
+          <param name="initial_value">${initial_positions['joint_a6']}</param>
         </state_interface>
       </joint>
-      <xacro:if value="${robot_description_package == 'kuka_lbr_iiwa_support'}">
+      <xacro:if value="${description_package == 'kuka_lbr_iiwa_support'}">
         <joint name="${prefix}joint_a7">
         <command_interface name="position">
@@ -92,5 +100,5 @@
         </command_interface>
         <state_interface name="position">
-          <param name="initial_value">0.0</param>
+          <param name="initial_value">${initial_positions['joint_a7']}</param>
         </state_interface>
         </joint>
