Commit message: Enable colors in robot visualization.

File: kuka_kr210_support/urdf/kr210r3100_macro.xacro (robot description, xacro)
@@ -1,4 +1,5 @@
 <?xml version="1.0"?>
 <robot xmlns:xacro="http://wiki.ros.org/xacro">
+  <xacro:include filename="$(find kuka_resources)/urdf/common_colours.xacro"/>
   <xacro:macro name="kuka_kr210r3100" params="prefix">
     <!-- links -->
@@ -14,6 +15,6 @@
           <mesh filename="file://$(find kuka_kr210_support)/meshes/kr210r3100/visual/base_link.stl" scale="0.001 0.001 0.001"/>
         </geometry>
-        <material name="">
-            <color rgba="0.75294 0.75294 0.75294 1"/>
+        <material name="colour_kuka_black">
+          <color rgba="${colour_kuka_black}"/>
         </material>
       </visual>
@@ -36,7 +37,7 @@
         <mesh filename="file://$(find kuka_kr210_support)/meshes/kr210r3100/visual/l1_1.stl" scale="0.001 0.001 0.001"/>
       </geometry>
-      <material name="">
-          <color rgba="0.75294 0.75294 0.75294 1"/>
-           </material>
+      <material name="colour_kuka_orange">
+        <color rgba="${colour_kuka_orange}"/>
+      </material>
     </visual>
     <collision>
@@ -58,7 +59,7 @@
         <mesh filename="file://$(find kuka_kr210_support)/meshes/kr210r3100/visual/l2_1.stl" scale="0.001 0.001 0.001"/>
       </geometry>
-      <material name="">
-          <color rgba="0.75294 0.75294 0.75294 1"/>
-           </material>
+      <material name="colour_kuka_orange">
+        <color rgba="${colour_kuka_orange}"/>
+      </material>
     </visual>
     <collision>
@@ -80,7 +81,7 @@
         <mesh filename="file://$(find kuka_kr210_support)/meshes/kr210r3100/visual/l3_1.stl" scale="0.001 0.001 0.001"/>
       </geometry>
-      <material name="">
-          <color rgba="0.75294 0.75294 0.75294 1"/>
-           </material>
+      <material name="colour_kuka_orange">
+        <color rgba="${colour_kuka_orange}"/>
+      </material>
     </visual>
     <collision>
@@ -102,7 +103,7 @@
         <mesh filename="file://$(find kuka_kr210_support)/meshes/kr210r3100/visual/l4_1.stl" scale="0.001 0.001 0.001"/>
       </geometry>
-      <material name="">
-          <color rgba="0.75294 0.75294 0.75294 1"/>
-           </material>
+      <material name="colour_kuka_orange">
+        <color rgba="${colour_kuka_orange}"/>
+      </material>
     </visual>
     <collision>
@@ -124,7 +125,7 @@
         <mesh filename="file://$(find kuka_kr210_support)/meshes/kr210r3100/visual/l5_1.stl" scale="0.001 0.001 0.001"/>
       </geometry>
-      <material name="">
-          <color rgba="0.75294 0.75294 0.75294 1"/>
-           </material>
+      <material name="colour_kuka_orange">
+        <color rgba="${colour_kuka_orange}"/>
+      </material>
     </visual>
     <collision>
@@ -134,6 +135,6 @@
       </geometry>
     </collision>
-        </link>
-        <link name="${prefix}link_6">
+  </link>
+  <link name="${prefix}link_6">
     <inertial>
       <origin xyz="0.02169435909842532 -1.3980071648605966e-05 5.2250469270931355e-05" rpy="0 0 0"/>
@@ -146,7 +147,7 @@
         <mesh filename="file://$(find kuka_kr210_support)/meshes/kr210r3100/visual/l6_1.stl" scale="0.001 0.001 0.001"/>
       </geometry>
-      <material name="">
-          <color rgba="0.75294 0.75294 0.75294 1"/>
-           </material>
+      <material name="colour_kuka_black">
+        <color rgba="${colour_kuka_black}"/>
+      </material>
     </visual>
     <collision>
@@ -156,5 +157,5 @@
       </geometry>
     </collision>
-        </link>
+  </link>
         <!-- This frame corresponds to the $TOOL coordinate system in KUKA KRC controllers. -->
         <link name="${prefix}flange"/>

Commit message: Introduced specific limits for pick place demo

File: kuka_kr210_support/urdf/kr210r3100_macro.xacro (robot description, xacro)
@@ -187,5 +187,5 @@
           <child link="${prefix}link_4"/>
           <axis xyz="1 0 0"/>
-          <limit lower="${radians(-350)}" upper="${radians(350)}" effort="0" velocity="${radians(136)}"/>
+          <limit lower="${radians(-60)}" upper="${radians(60)}" effort="0" velocity="${radians(136)}"/>
       </joint>
       <joint name="${prefix}joint_a5" type="revolute">
@@ -201,5 +201,5 @@
           <child link="${prefix}link_6"/>
           <axis xyz="-1 0 0"/>
-          <limit lower="${radians(-350)}" upper="${radians(350)}" effort="0" velocity="${radians(206)}"/>
+          <limit lower="${radians(-215)}" upper="${radians(250)}" effort="0" velocity="${radians(206)}"/>
       </joint>
       <joint name="${prefix}link_6-flange" type="fixed">

Commit message: Adjust joint limits for kr 210 r3100-2 in urdf

File: kuka_kr210_support/urdf/kr210r3100_macro.xacro (robot description, xacro)
@@ -173,5 +173,5 @@
           <child link="${prefix}link_2"/>
           <axis xyz="0 1 0"/>
-          <limit lower="${radians(-140)}" upper="${radians(-14)}" effort="0" velocity="${radians(94)}"/>
+          <limit lower="${radians(-140)}" upper="${radians(-5)}" effort="0" velocity="${radians(94)}"/>
       </joint>
       <joint name="${prefix}joint_a3" type="revolute">
@@ -187,5 +187,5 @@
           <child link="${prefix}link_4"/>
           <axis xyz="1 0 0"/>
-          <limit lower="${radians(-60)}" upper="${radians(60)}" effort="0" velocity="${radians(136)}"/>
+          <limit lower="${radians(-350)}" upper="${radians(350)}" effort="0" velocity="${radians(136)}"/>
       </joint>
       <joint name="${prefix}joint_a5" type="revolute">
@@ -201,5 +201,5 @@
           <child link="${prefix}link_6"/>
           <axis xyz="-1 0 0"/>
-          <limit lower="${radians(-215)}" upper="${radians(250)}" effort="0" velocity="${radians(206)}"/>
+          <limit lower="${radians(-350)}" upper="${radians(350)}" effort="0" velocity="${radians(206)}"/>
       </joint>
       <joint name="${prefix}link_6-flange" type="fixed">

Commit message: Fix orientation of joint_a4

File: kuka_kr210_support/urdf/kr210r3100_macro.xacro (robot description, xacro)
@@ -186,5 +186,5 @@
           <parent link="${prefix}link_3"/>
           <child link="${prefix}link_4"/>
-          <axis xyz="1 0 0"/>
+          <axis xyz="-1 0 0"/>
           <limit lower="${radians(-350)}" upper="${radians(350)}" effort="0" velocity="${radians(136)}"/>
       </joint>
